File: mippe_base/mippe_base.sch (EAGLE design)
At the start: 17 parts, among them IC1 ATMEGA168PROUND, SW1 BTN-PTS810

Commit message: Finish burnin and mippe controller
Parts:
- added D2: RED, scono:LED0603
- added J8: (no value), scono:CONN_041X04_NO_SILK
- added J9: BURNIN, scono:BURNIN
- added R3: 330R, scono:R-US_R0603
- R2: value (none) -> 330R
- Y1: value (none) -> 16MHz
Connections:
- removed net DTR: J1.6
- new net N$2: D2.A, R3.2
- net 3.3V: now also J9.3.3V, R3.1
- net GND: now also D2.C, J9.GND
- net GPIO3: now also J8.4
- net GPIO4: now also J8.3
- net GPIO5: now also J8.2
- net GPIO6: now also J8.1
- net MISO: now also J9.MISO
- net MOSI: now also J9.MOSI
- net RST: now also J1.6
- net SCK: now also J9.SCK
- net SS: now also J9.SS
Changed lines of the file:
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@@
 <part name="IC1" library="scono" deviceset="ATMEGA168*P" device="ROUND"/>
 <part name="R1" library="scono" deviceset="R-US_" device="R0603"/>
-<part name="R2" library="scono" deviceset="R-US_" device="R0603"/>
+<part name="R2" library="scono" deviceset="R-US_" device="R0603" value="330R"/>
 <part name="D1" library="scono" deviceset="LED" device="0603"/>
 <part name="SUPPLY1" library="scono" deviceset="GND" device=""/>
@@
 <part name="SW1" library="scono" deviceset="BTN-PTS810" device=""/>
 <part name="SUPPLY6" library="scono" deviceset="GND" device=""/>
-<part name="Y1" library="scono" deviceset="CRYSTAL" device=""/>
+<part name="Y1" library="scono" deviceset="CRYSTAL" device="" value="16MHz"/>
 <part name="C3" library="scono" deviceset="CAP" device="0603-CAP" value="18pF"/>
 <part name="C4" library="scono" deviceset="CAP" device="0603-CAP" value="18pF"/>
@@
 <part name="J6" library="scono" deviceset="CONN_04" device="1X04_NO_SILK" package3d_urn="urn:adsk.eagle:package:38094/1"/>
 <part name="J7" library="scono" deviceset="CONN_02" device="1X02_NO_SILK" package3d_urn="urn:adsk.eagle:package:38051/1"/>
+<part name="J8" library="scono" deviceset="CONN_04" device="1X04_NO_SILK" package3d_urn="urn:adsk.eagle:package:38094/1"/>
+<part name="R3" library="scono" deviceset="R-US_" device="R0603" value="330R"/>
+<part name="D2" library="scono" deviceset="LED" device="0603" value="RED"/>
+<part name="SUPPLY10" library="scono" deviceset="GND" device=""/>
+<part name="U$7" library="scono" deviceset="3.3V" device=""/>
+<part name="J9" library="scono" deviceset="BURNIN" device=""/>
+<part name="U$8" library="scono" deviceset="3.3V" device=""/>
+<part name="SUPPLY11" library="scono" deviceset="GND" device=""/>
 </parts>
 <sheets>
@@
 <attribute name="NAME" x="205.74" y="109.728" size="1.778" layer="95" font="vector"/>
 </instance>
+<instance part="J8" gate="G$1" x="210.82" y="86.36" smashed="yes">
+<attribute name="VALUE" x="205.74" y="78.994" size="1.778" layer="96" font="vector"/>
+<attribute name="NAME" x="205.74" y="94.488" size="1.778" layer="95" font="vector"/>
+</instance>
+<instance part="R3" gate="G$1" x="101.6" y="157.48" smashed="yes" rot="R270">
+<attribute name="NAME" x="102.87" y="162.56" size="1.016" layer="95" rot="R270"/>
+<attribute name="VALUE" x="100.33" y="162.56" size="1.016" layer="96" rot="R270" align="top-left"/>
+</instance>
+<instance part="D2" gate="G$1" x="101.6" y="152.4" smashed="yes">
+<attribute name="NAME" x="98.171" y="147.828" size="1.778" layer="95" font="vector" rot="R90"/>
+<attribute name="VALUE" x="103.505" y="147.828" size="1.778" layer="96" font="vector" rot="R90" align="top-left"/>
+</instance>
+<instance part="SUPPLY10" gate="GND" x="101.6" y="144.78" smashed="yes">
+<attribute name="VALUE" x="100.33" y="142.24" size="1.016" layer="96"/>
+</instance>
+<instance part="U$7" gate="G$1" x="101.6" y="162.56" smashed="yes">
+<attribute name="VALUE" x="100.33" y="166.37" size="1.778" layer="96"/>
+</instance>
+<instance part="J9" gate="G$1" x="55.88" y="157.48" smashed="yes">
+<attribute name="NAME" x="48.26" y="167.64" size="1.778" layer="94" align="top-left"/>
+</instance>
+<instance part="U$8" gate="G$1" x="45.72" y="162.56" smashed="yes" rot="R90">
+<attribute name="VALUE" x="41.91" y="161.29" size="1.778" layer="96" rot="R90"/>
+</instance>
+<instance part="SUPPLY11" gate="GND" x="43.18" y="149.86" smashed="yes" rot="R270">
+<attribute name="VALUE" x="40.64" y="151.13" size="1.016" layer="96" rot="R270"/>
+</instance>
 </instances>
 <busses>
@@
 <label x="180.34" y="152.4" size="1.778" layer="95"/>
 </segment>
+<segment>
+<pinref part="D2" gate="G$1" pin="C"/>
+<pinref part="SUPPLY10" gate="GND" pin="GND"/>
+</segment>
+<segment>
+<pinref part="J9" gate="G$1" pin="GND"/>
+<pinref part="SUPPLY11" gate="GND" pin="GND"/>
+</segment>
 </net>
 <net name="3.3V" class="0">
@@
 <label x="180.34" y="157.48" size="1.778" layer="95"/>
 </segment>
+<segment>
+<pinref part="R3" gate="G$1" pin="1"/>
+<pinref part="U$7" gate="G$1" pin="3.3V"/>
+</segment>
+<segment>
+<pinref part="J9" gate="G$1" pin="3.3V"/>
+<pinref part="U$8" gate="G$1" pin="3.3V"/>
+</segment>
 </net>
 <net name="SCL" class="0">
@@
 <label x="152.4" y="91.44" size="1.778" layer="95"/>
 </segment>
+<segment>
+<pinref part="J8" gate="G$1" pin="4"/>
+<wire x1="215.9" y1="91.44" x2="218.44" y2="91.44" width="0.1524" layer="91"/>
+<label x="218.44" y="91.44" size="1.778" layer="95"/>
+</segment>
 </net>
 <net name="GPIO4" class="0">
@@
 <label x="152.4" y="88.9" size="1.778" layer="95"/>
 </segment>
+<segment>
+<pinref part="J8" gate="G$1" pin="3"/>
+<wire x1="215.9" y1="88.9" x2="218.44" y2="88.9" width="0.1524" layer="91"/>
+<label x="218.44" y="88.9" size="1.778" layer="95"/>
+</segment>
 </net>
 <net name="GPIO5" class="0">
@@
 <label x="152.4" y="86.36" size="1.778" layer="95"/>
 </segment>
+<segment>
+<pinref part="J8" gate="G$1" pin="2"/>
+<wire x1="215.9" y1="86.36" x2="218.44" y2="86.36" width="0.1524" layer="91"/>
+<label x="218.44" y="86.36" size="1.778" layer="95"/>
+</segment>
 </net>
 <net name="GPIO6" class="0">
@@
 <wire x1="142.24" y1="81.28" x2="152.4" y2="81.28" width="0.1524" layer="91"/>
 <label x="152.4" y="81.28" size="1.778" layer="95"/>
+</segment>
+<segment>
+<pinref part="J8" gate="G$1" pin="1"/>
+<wire x1="215.9" y1="83.82" x2="218.44" y2="83.82" width="0.1524" layer="91"/>
+<label x="218.44" y="83.82" size="1.778" layer="95"/>
 </segment>
 </net>
@@
 <label x="180.34" y="134.62" size="1.778" layer="95"/>
 </segment>
+<segment>
+<pinref part="J9" gate="G$1" pin="SS"/>
+<wire x1="45.72" y1="152.4" x2="38.1" y2="152.4" width="0.1524" layer="91"/>
+<label x="30.48" y="152.4" size="1.778" layer="95"/>
+</segment>
 </net>
 <net name="MOSI" class="0">
@@
 <label x="180.34" y="137.16" size="1.778" layer="95"/>
 </segment>
+<segment>
+<pinref part="J9" gate="G$1" pin="MOSI"/>
+<wire x1="38.1" y1="154.94" x2="45.72" y2="154.94" width="0.1524" layer="91"/>
+<label x="30.48" y="154.94" size="1.778" layer="95"/>
+</segment>
 </net>
 <net name="MISO" class="0">
@@
 <label x="180.34" y="139.7" size="1.778" layer="95"/>
 </segment>
+<segment>
+<pinref part="J9" gate="G$1" pin="MISO"/>
+<wire x1="45.72" y1="157.48" x2="38.1" y2="157.48" width="0.1524" layer="91"/>
+<label x="30.48" y="157.48" size="1.778" layer="95"/>
+</segment>
 </net>
 <net name="SCK" class="0">
@@
 <wire x1="177.8" y1="142.24" x2="180.34" y2="142.24" width="0.1524" layer="91"/>
 <label x="180.34" y="142.24" size="1.778" layer="95"/>
+</segment>
+<segment>
+<pinref part="J9" gate="G$1" pin="SCK"/>
+<wire x1="45.72" y1="160.02" x2="38.1" y2="160.02" width="0.1524" layer="91"/>
+<label x="30.48" y="160.02" size="1.778" layer="95"/>
 </segment>
 </net>
@@
 <label x="81.28" y="129.54" size="1.778" layer="95"/>
 </segment>
+<segment>
+<pinref part="J1" gate="G$1" pin="6"/>
+<wire x1="177.8" y1="165.1" x2="180.34" y2="165.1" width="0.1524" layer="91"/>
+<label x="180.34" y="165.1" size="1.778" layer="95"/>
+</segment>
 </net>
 <net name="N$3" class="0">
@@
 </segment>
 </net>
-<net name="DTR" class="0">
-<segment>
-<pinref part="J1" gate="G$1" pin="6"/>
-<wire x1="177.8" y1="165.1" x2="180.34" y2="165.1" width="0.1524" layer="91"/>
-<label x="180.34" y="165.1" size="1.778" layer="95"/>
-</segment>
-</net>
 <net name="CTS" class="0">
 <segment>
@@
 </segment>
 </net>
+<net name="N$2" class="0">
+<segment>
+<pinref part="R3" gate="G$1" pin="2"/>
+<pinref part="D2" gate="G$1" pin="A"/>
+</segment>
+</net>
