File: mippe_base_v2/mippe_base_v2.brd (EAGLE design)
At the start: 27 x 31.5 mm, 21 parts, among them J9 BURNIN, SW1 BTN-PTS810, U1 ATMEGA328P-AUR, Y1 16MHz

Commit message: fix rst and flip conn
Parts:
- added C5: 0.1uF, scono:0603-CAP
Connections:
- new net N$3: C5.2, J1.1
- net 3.3V: now also J1.4; no longer J1.3
- net CTS: now also J1.5; no longer J1.2
- net GND: now also J1.6; no longer J1.1
- net RST: now also C5.1; no longer J1.6
- net RX: now also J1.3; no longer J1.4
- net TX: now also J1.2; no longer J1.5
Routing:
- net N$3: track 0.00 -> 10.2 mm
- net 3.3V: track 14.4 -> 9.31 mm
- net RX: track 35.9 -> 31.9 mm, vias 3 -> 2
- net GND: track 33.5 -> 37.5 mm
- net TX: track 35.4 -> 31.6 mm, vias 3 -> 2
- net RST: track 22.7 -> 24.9 mm, vias 0 -> 1
Other:
- board text added: "MIPPE Rev C"
- board text removed: "MIPPE Rev B"
Changed lines of the file:
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@@
 <wire x1="0" y1="5" x2="0" y2="29.75" width="0" layer="20"/>
 <text x="3.75" y="27.75" size="1" layer="21" font="vector">MIPPE
-Rev B</text>
+Rev C</text>
 <text x="23.25" y="28" size="1.5" layer="22" font="vector" rot="MR270">Arias Research Group
 ATMega328P Custom</text>
@@
 <attribute name="VALUE" x="17.45" y="30.2" size="1.2" layer="27" font="vector" rot="R270"/>
 </element>
+<element name="C5" library="scono" package="0603-CAP" value="0.1uF" x="15.25" y="10.25" smashed="yes" rot="R180">
+<attribute name="NAME" x="16.52" y="9.488" size="0.508" layer="25" font="vector" ratio="10" rot="R180"/>
+<attribute name="PIE-INT-REF-NUM" value="CAPACITOR-GENERIC" x="15.25" y="10.25" size="1.778" layer="27" rot="R180" display="off"/>
+<attribute name="VALUE" x="16.52" y="11.647" size="0.508" layer="27" font="vector" rot="R180"/>
+</element>
 </elements>
 <signals>
@@
 <contactref element="J4" pad="2"/>
 <contactref element="J4" pad="1"/>
-<contactref element="J1" pad="1"/>
 <contactref element="D2" pad="C"/>
 <contactref element="J9" pad="GND"/>
@@
 <wire x1="3.6" y1="21.4" x2="3.5" y2="21.5" width="0.2" layer="1"/>
 <via x="3.5" y="21.5" extent="1-16" drill="0.4"/>
+<contactref element="J1" pad="6"/>
+<wire x1="9" y1="14.5" x2="8.25" y2="14.5" width="0.2" layer="1"/>
+<wire x1="7" y1="15.75" x2="5.5" y2="15.75" width="0.2" layer="1"/>
+<wire x1="8.25" y1="14.5" x2="7" y2="15.75" width="0.2" layer="1"/>
 </signal>
 <signal name="3.3V">
@@
 <contactref element="J3" pad="2"/>
 <contactref element="J3" pad="1"/>
-<contactref element="J1" pad="3"/>
 <contactref element="R3" pad="1"/>
 <contactref element="J9" pad="3.3V"/>
@@
 <wire x1="12.98" y1="4.97" x2="13.03" y2="4.97" width="0.2" layer="16"/>
 <wire x1="13.03" y1="4.97" x2="14" y2="4" width="0.2" layer="16"/>
-<via x="14" y="4" extent="1-16" drill="0.4"/>
-<wire x1="14" y1="4" x2="13.91" y2="4" width="0.2" layer="1"/>
-<wire x1="13.91" y1="4" x2="10.41" y2="7.5" width="0.2" layer="1"/>
+<contactref element="J1" pad="4"/>
+<via x="14" y="4" extent="1-16" drill="0.381"/>
 </signal>
 <signal name="SCL">
@@
 </signal>
 <signal name="RX">
-<contactref element="J1" pad="4"/>
 <contactref element="J7" pad="1"/>
 <contactref element="U1" pad="30"/>
@@
 <wire x1="12.75" y1="19.5" x2="13.0728375" y2="19.5" width="0.2" layer="16"/>
 <wire x1="13.0728375" y1="19.5" x2="13.7284375" y2="18.8444" width="0.2" layer="16"/>
-<wire x1="12.95" y1="7.5" x2="10.7" y2="9.75" width="0.2" layer="1"/>
-<wire x1="10.7" y1="9.75" x2="9" y2="9.75" width="0.2" layer="1"/>
-<wire x1="7.75" y1="11" x2="9" y2="9.75" width="0.2" layer="1"/>
-<wire x1="7.75" y1="11" x2="7.75" y2="15.25" width="0.2" layer="1"/>
-<wire x1="7.75" y1="15.25" x2="7" y2="16" width="0.2" layer="1"/>
-<via x="7" y="16" extent="1-16" drill="0.4"/>
-<wire x1="7" y1="16" x2="7" y2="17.75" width="0.2" layer="16"/>
-<wire x1="7" y1="17.75" x2="9.25" y2="20" width="0.2" layer="16"/>
-<via x="9.25" y="20" extent="1-16" drill="0.4"/>
 <wire x1="12.75" y1="19.5" x2="10.6771625" y2="19.5" width="0.2" layer="1"/>
 <wire x1="10.6771625" y1="19.5" x2="10.5215625" y2="19.3444" width="0.2" layer="1"/>
-<wire x1="10.5215625" y1="19.3444" x2="9.9056" y2="19.3444" width="0.2" layer="1"/>
-<wire x1="9.9056" y1="19.3444" x2="9.25" y2="20" width="0.2" layer="1"/>
+<wire x1="10.5215625" y1="19.3444" x2="10" y2="19.3444" width="0.2" layer="1"/>
+<wire x1="10" y1="19.3444" x2="9.9056" y2="19.3444" width="0.2" layer="1"/>
 <wire x1="19.157225" y1="18.8444" x2="20.314025" y2="17.6876" width="0.2" layer="16"/>
 <wire x1="22.9524" y1="17.6876" x2="24.9" y2="15.74" width="0.2" layer="16"/>
 <wire x1="20.314025" y1="17.6876" x2="22.9524" y2="17.6876" width="0.2" layer="16"/>
 <wire x1="13.7284375" y1="18.8444" x2="19.157225" y2="18.8444" width="0.2" layer="16"/>
+<contactref element="J1" pad="3"/>
+<wire x1="10" y1="19.3444" x2="9.9056" y2="19.3444" width="0.2" layer="1"/>
+<wire x1="9.9056" y1="19.3444" x2="9.774678125" y2="19.475321875" width="0.2" layer="1"/>
+<via x="9.774678125" y="19.475321875" extent="1-16" drill="0.381"/>
+<wire x1="9.774678125" y1="19.475321875" x2="8.25" y2="17.95064375" width="0.2" layer="16"/>
+<wire x1="8.25" y1="17.95064375" x2="8.25" y2="15.25" width="0.2" layer="16"/>
+<wire x1="8.25" y1="15.25" x2="8.25" y2="9.66" width="0.2" layer="16"/>
+<wire x1="8.25" y1="9.66" x2="10.41" y2="7.5" width="0.2" layer="16"/>
 </signal>
 <signal name="TX">
-<contactref element="J1" pad="5"/>
 <contactref element="J7" pad="2"/>
 <contactref element="U1" pad="31"/>
@@
 <wire x1="20.22" y1="18.28" x2="24.9" y2="18.28" width="0.2" layer="16"/>
 <wire x1="19" y1="19.5" x2="20.22" y2="18.28" width="0.2" layer="16"/>
-<wire x1="15.49" y1="7.5" x2="12.49" y2="10.5" width="0.2" layer="1"/>
-<wire x1="12.49" y1="10.5" x2="9" y2="10.5" width="0.2" layer="1"/>
-<wire x1="9" y1="10.5" x2="8.25" y2="11.25" width="0.2" layer="1"/>
-<via x="8.25" y="16" extent="1-16" drill="0.4"/>
-<wire x1="8.25" y1="11.25" x2="8.25" y2="16" width="0.2" layer="1"/>
-<wire x1="8.25" y1="16" x2="8.25" y2="18" width="0.2" layer="16"/>
-<wire x1="8.25" y1="18" x2="10.25" y2="20" width="0.2" layer="16"/>
-<via x="10.25" y="20" extent="1-16" drill="0.4"/>
-<wire x1="10.25" y1="20" x2="12.3228375" y2="20" width="0.2" layer="1"/>
-<wire x1="12.3228375" y1="20" x2="12.4784375" y2="20.1556" width="0.2" layer="1"/>
+<wire x1="12.4784375" y1="20.1556" x2="12.3228375" y2="20" width="0.2" layer="1"/>
 <wire x1="13.4784375" y1="19.8444" x2="13.6556" y2="19.8444" width="0.2" layer="1"/>
 <wire x1="13.6556" y1="19.8444" x2="14" y2="19.5" width="0.2" layer="1"/>
 <wire x1="12.4784375" y1="20.1556" x2="13.1672375" y2="20.1556" width="0.2" layer="1"/>
 <wire x1="13.1672375" y1="20.1556" x2="13.4784375" y2="19.8444" width="0.2" layer="1"/>
+<contactref element="J1" pad="2"/>
+<via x="9" y="20" extent="1-16" drill="0.381"/>
+<wire x1="12.3228375" y1="20" x2="10.1278125" y2="20" width="0.2" layer="1"/>
+<wire x1="10.1278125" y1="20" x2="10.0317875" y2="20.096025" width="0.2" layer="1"/>
+<wire x1="10.0317875" y1="20.096025" x2="9.517575" y2="20.096025" width="0.2" layer="1"/>
+<wire x1="9.517575" y1="20.096025" x2="9.42155" y2="20" width="0.2" layer="1"/>
+<wire x1="9.42155" y1="20" x2="9" y2="20" width="0.2" layer="1"/>
+<wire x1="9" y1="20" x2="7.5" y2="18.5" width="0.2" layer="16"/>
+<wire x1="7.5" y1="7.87" x2="7.87" y2="7.5" width="0.2" layer="16"/>
+<wire x1="7.5" y1="18.5" x2="7.5" y2="7.87" width="0.2" layer="16"/>
 </signal>
 <signal name="GPIO1">
@@
 <contactref element="SW1" pad="3"/>
 <contactref element="SW1" pad="4"/>
-<contactref element="J1" pad="6"/>
 <contactref element="U1" pad="29"/>
 <contactref element="J9" pad="RST"/>
 <wire x1="18.06" y1="2.43" x2="19.25" y2="3.62" width="0.2" layer="16"/>
-<wire x1="19.25" y1="6.28" x2="18.03" y2="7.5" width="0.2" layer="16"/>
-<wire x1="19.25" y1="3.62" x2="19.25" y2="6.28" width="0.2" layer="16"/>
-<wire x1="18.03" y1="7.5" x2="18.03" y2="10.62" width="0.2" layer="1"/>
 <wire x1="18.03" y1="10.62" x2="18.095" y2="10.685" width="0.2" layer="1"/>
 <wire x1="12.15" y1="18.07" x2="12.4226" y2="17.7974" width="0.2" layer="1"/>
@@
 <wire x1="15.75" y1="13.85" x2="14.5" y2="15.1" width="0.2" layer="1"/>
 <wire x1="14.5" y1="15.1" x2="14.5" y2="16.75" width="0.2" layer="1"/>
-</signal>
-<signal name="CTS">
-<contactref element="J1" pad="2"/>
+<contactref element="C5" pad="1"/>
+<wire x1="19.25" y1="9.25" x2="19" y2="9.5" width="0.2" layer="16"/>
+<via x="19" y="9.5" extent="1-16" drill="0.381"/>
+<wire x1="19" y1="9.5" x2="18.03" y2="10.47" width="0.2" layer="1"/>
+<wire x1="18.03" y1="10.47" x2="18.03" y2="10.62" width="0.2" layer="1"/>
+<wire x1="19.25" y1="3.62" x2="19.25" y2="9.25" width="0.2" layer="16"/>
+<wire x1="18.095" y1="10.685" x2="17.66" y2="10.25" width="0.2" layer="1"/>
+<wire x1="17.66" y1="10.25" x2="16.1" y2="10.25" width="0.2" layer="1"/>
 </signal>
 <signal name="N$2">
@@
 <wire x1="19.8" y1="25.05" x2="21.25" y2="26.5" width="0.2" layer="1"/>
 </signal>
+<signal name="CTS">
+<contactref element="J1" pad="5"/>
+</signal>
+<signal name="N$3">
+<contactref element="J1" pad="1"/>
+<contactref element="C5" pad="2"/>
+<wire x1="5.33" y1="7.5" x2="8.08" y2="10.25" width="0.2" layer="1"/>
+<wire x1="8.08" y1="10.25" x2="14.4" y2="10.25" width="0.2" layer="1"/>
+</signal>
 </signals>
