File: mippe_base_32u4/mippe_32u4.sch (EAGLE design)
At the start: 27 parts, among them J2 USB, SW1 BTN-PTS810, U1 ATMEGA32U4-XUMU, U2 AZ1117EH-3.3TRG1, Y1 16MHz

Commit message: Progress on layout
Parts:
- removed C12, C8: 1uF, scono:CAP0603-CAP
- removed U2: AZ1117EH-3.3TRG1, scono:AZ1117EH-3.3TRG1
- U1: device SmartPrj:ATMEGA32U4-XUMU -> scono:ATMEGA32U4-XUMU
- Z1, Z2: device varistor:VARISTORCN0603 -> scono:VARISTOR
Connections:
- removed net 3.3V: C12.2, U2.OUT
- net 5V: no longer C8.2, U2.IN
- net GND: no longer C12.1, C8.1, U2.ADJ/GND
Changed lines of the file:
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@@
 </classes>
 <parts>
-<part name="Z1" library="varistor" deviceset="VARISTOR" device="CN0603" value="CG0603MLC-05E"/>
-<part name="Z2" library="varistor" deviceset="VARISTOR" device="CN0603" value="CG0603MLC-05E"/>
-<part name="U1" library="SmartPrj" deviceset="ATMEGA32U4-XU" device="MU"/>
+<part name="Z1" library="scono" deviceset="VARISTOR" device="" value="CG0603MLC-05E"/>
+<part name="Z2" library="scono" deviceset="VARISTOR" device="" value="CG0603MLC-05E"/>
+<part name="U1" library="scono" deviceset="ATMEGA32U4-XU" device="MU"/>
 <part name="FRAME2" library="scono" deviceset="FRAME_SCHEMATIC" device="">
 <attribute name="AUTHOR" value="S.Ono"/>
@@
 </part>
 <part name="C10" library="scono" deviceset="CAP" device="0603-CAP" value="1uF"/>
-<part name="U2" library="scono" deviceset="AZ1117EH-3.3TRG1" device=""/>
-<part name="U$1" library="scono" deviceset="5V" device=""/>
-<part name="U$2" library="scono" deviceset="3.3V" device=""/>
-<part name="SUPPLY3" library="scono" deviceset="GND" device=""/>
-<part name="C8" library="scono" deviceset="CAP" device="0603-CAP" value="1uF"/>
-<part name="C12" library="scono" deviceset="CAP" device="0603-CAP" value="1uF"/>
-<part name="SUPPLY4" library="scono" deviceset="GND" device=""/>
 <part name="U$3" library="scono" deviceset="5V" device=""/>
 <part name="U$4" library="scono" deviceset="5V" device=""/>
@@
 <attribute name="VALUE" x="-294.64" y="-135.89" size="1.016" layer="96" rot="R90"/>
 </instance>
-<instance part="U2" gate="G$1" x="-350.52" y="-50.8" smashed="yes">
-<attribute name="NAME" x="-358.14941875" y="-45.71371875" size="1.7802" layer="95"/>
-<attribute name="VALUE" x="-358.147440625" y="-58.427440625" size="1.779740625" layer="96"/>
-</instance>
-<instance part="U$1" gate="G$1" x="-363.22" y="-43.18" smashed="yes">
-<attribute name="VALUE" x="-364.49" y="-39.37" size="1.778" layer="96"/>
-</instance>
-<instance part="U$2" gate="G$1" x="-330.2" y="-43.18" smashed="yes">
-<attribute name="VALUE" x="-331.47" y="-39.37" size="1.778" layer="96"/>
-</instance>
-<instance part="SUPPLY3" gate="GND" x="-330.2" y="-55.88" smashed="yes">
-<attribute name="VALUE" x="-331.47" y="-58.42" size="1.016" layer="96"/>
-</instance>
-<instance part="C8" gate="G$1" x="-363.22" y="-50.8" smashed="yes" rot="MR90">
-<attribute name="NAME" x="-365.76" y="-48.26" size="1.778" layer="95" rot="MR90"/>
-<attribute name="VALUE" x="-363.22" y="-48.26" size="1.778" layer="96" rot="MR90"/>
-</instance>
-<instance part="C12" gate="G$1" x="-330.2" y="-50.8" smashed="yes" rot="R90">
-<attribute name="NAME" x="-326.898" y="-48.895" size="1.778" layer="95" rot="R270"/>
-<attribute name="VALUE" x="-335.153" y="-49.149" size="1.778" layer="96" rot="R270"/>
-</instance>
-<instance part="SUPPLY4" gate="GND" x="-363.22" y="-55.88" smashed="yes">
-<attribute name="VALUE" x="-364.49" y="-58.42" size="1.016" layer="96"/>
-</instance>
 <instance part="U$3" gate="G$1" x="-256.54" y="-68.58" smashed="yes">
 <attribute name="VALUE" x="-257.81" y="-64.77" size="1.778" layer="96"/>
@@
 <nets>
 <net name="GND" class="2">
-<segment>
-<pinref part="U2" gate="G$1" pin="ADJ/GND"/>
-<pinref part="SUPPLY3" gate="GND" pin="GND"/>
-<wire x1="-340.36" y1="-53.34" x2="-330.2" y2="-53.34" width="0.1524" layer="91"/>
-<pinref part="C12" gate="G$1" pin="1"/>
-<junction x="-330.2" y="-53.34"/>
-</segment>
-<segment>
-<pinref part="C8" gate="G$1" pin="1"/>
-<pinref part="SUPPLY4" gate="GND" pin="GND"/>
-</segment>
 <segment>
 <pinref part="Z1" gate="G$1" pin="2"/>
@@
 <pinref part="SUPPLY5" gate="GND" pin="GND"/>
 <pinref part="C9" gate="G$1" pin="1"/>
+<junction x="-309.88" y="-139.7"/>
 </segment>
 <segment>
@@
 <net name="5V" class="0">
 <segment>
-<pinref part="U$1" gate="G$1" pin="5V"/>
-<wire x1="-363.22" y1="-43.18" x2="-363.22" y2="-48.26" width="0.1524" layer="91"/>
-<pinref part="U2" gate="G$1" pin="IN"/>
-<wire x1="-363.22" y1="-48.26" x2="-360.68" y2="-48.26" width="0.1524" layer="91"/>
-<pinref part="C8" gate="G$1" pin="2"/>
-<junction x="-363.22" y="-48.26"/>
-</segment>
-<segment>
 <wire x1="-309.88" y1="-132.08" x2="-309.88" y2="-129.54" width="0.1524" layer="91"/>
 <wire x1="-309.88" y1="-129.54" x2="-309.88" y2="-124.46" width="0.1524" layer="91"/>
@@
 <pinref part="U$4" gate="G$1" pin="5V"/>
 <pinref part="C9" gate="G$1" pin="2"/>
+<junction x="-309.88" y="-129.54"/>
 </segment>
 <segment>
@@
 <pinref part="R6" gate="G$1" pin="2"/>
 <wire x1="-256.54" y1="-76.2" x2="-256.54" y2="-78.74" width="0.1524" layer="91"/>
-</segment>
-</net>
-<net name="3.3V" class="0">
-<segment>
-<pinref part="U2" gate="G$1" pin="OUT"/>
-<wire x1="-340.36" y1="-48.26" x2="-330.2" y2="-48.26" width="0.1524" layer="91"/>
-<pinref part="U$2" gate="G$1" pin="3.3V"/>
-<wire x1="-330.2" y1="-48.26" x2="-330.2" y2="-43.18" width="0.1524" layer="91"/>
-<pinref part="C12" gate="G$1" pin="2"/>
-<junction x="-330.2" y="-48.26"/>
 </segment>
 </net>
@@
 <wire x1="20.32" y1="106.68" x2="25.4" y2="106.68" width="0.1524" layer="91"/>
 <label x="22.86" y="109.22" size="1.27" layer="95"/>
+<junction x="25.4" y="106.68"/>
 </segment>
 </net>
@@
 <wire x1="10.16" y1="106.68" x2="15.24" y2="106.68" width="0.1524" layer="91"/>
 <label x="7.62" y="109.22" size="1.27" layer="95"/>
+<junction x="10.16" y="106.68"/>
 </segment>
 </net>
@@
 <pinref part="C11" gate="G$1" pin="1"/>
 <wire x1="104.14" y1="81.28" x2="104.14" y2="76.2" width="0.1524" layer="91"/>
+<label x="104.14" y="73.66" size="1.778" layer="95"/>
 </segment>
 </net>
@@
 <pinref part="U1" gate="G$1" pin="VBUS"/>
 <pinref part="U$8" gate="G$1" pin="5V"/>
-</segment>
-<segment>
-<wire x1="114.3" y1="96.52" x2="116.84" y2="96.52" width="0.1524" layer="91"/>
-<wire x1="116.84" y1="83.82" x2="114.3" y2="83.82" width="0.1524" layer="91"/>
-<wire x1="114.3" y1="83.82" x2="114.3" y2="96.52" width="0.1524" layer="91"/>
-<wire x1="114.3" y1="104.14" x2="114.3" y2="96.52" width="0.1524" layer="91"/>
-<junction x="114.3" y="96.52"/>
-<pinref part="U1" gate="G$1" pin="UVCC"/>
-<pinref part="U1" gate="G$1" pin="VCC"/>
 </segment>
 <segment>
@@
 <pinref part="C1" gate="G$1" pin="2"/>
 <wire x1="101.6" y1="142.24" x2="101.6" y2="139.7" width="0.1524" layer="91"/>
+<junction x="91.44" y="142.24"/>
 </segment>
 <segment>
@@
 <wire x1="60.96" y1="101.6" x2="101.6" y2="101.6" width="0.1524" layer="91"/>
 <wire x1="101.6" y1="101.6" x2="101.6" y2="106.68" width="0.1524" layer="91"/>
-<wire x1="116.84" y1="104.14" x2="111.76" y2="104.14" width="0.1524" layer="91"/>
+<wire x1="116.84" y1="104.14" x2="114.3" y2="104.14" width="0.1524" layer="91"/>
+<wire x1="114.3" y1="104.14" x2="111.76" y2="104.14" width="0.1524" layer="91"/>
 <wire x1="111.76" y1="104.14" x2="111.76" y2="106.68" width="0.1524" layer="91"/>
 <junction x="101.6" y="106.68"/>
@@
 <wire x1="86.36" y1="106.68" x2="96.52" y2="106.68" width="0.1524" layer="91"/>
 <pinref part="C5" gate="G$1" pin="2"/>
-</segment>
-<segment>
+<wire x1="114.3" y1="96.52" x2="116.84" y2="96.52" width="0.1524" layer="91"/>
+<wire x1="116.84" y1="83.82" x2="114.3" y2="83.82" width="0.1524" layer="91"/>
+<wire x1="114.3" y1="83.82" x2="114.3" y2="96.52" width="0.1524" layer="91"/>
+<wire x1="114.3" y1="104.14" x2="114.3" y2="96.52" width="0.1524" layer="91"/>
+<junction x="114.3" y="96.52"/>
+<pinref part="U1" gate="G$1" pin="UVCC"/>
+<pinref part="U1" gate="G$1" pin="VCC"/>
+<junction x="114.3" y="104.14"/>
+</segment>
+<segment>

Commit message: blah
Connections:
- net D+ renamed D_P
- net D- renamed D_N
- net RD+ renamed RD_P
- net RD- renamed RD_N
Changed lines of the file:
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@@
 </variantdefs>
 <classes>
-<class number="0" name="default" width="0.254" drill="0.499">
-<clearance class="0" value="0.254"/>
+<class number="0" name="default" width="0.1524" drill="0.381">
+<clearance class="0" value="0.1524"/>
 </class>
 <class number="1" name="power" width="0.254" drill="0.499">
+<clearance class="0" value="0.1524"/>
 <clearance class="1" value="0.254"/>
 </class>
 <class number="2" name="gnd" width="0.254" drill="0.499">
+<clearance class="0" value="0.1524"/>
+<clearance class="1" value="0.1524"/>
 <clearance class="2" value="0.254"/>
 </class>
 <class number="3" name="usbvcc" width="0.254" drill="0.499">
+<clearance class="0" value="0.1524"/>
+<clearance class="1" value="0.1524"/>
+<clearance class="2" value="0.1524"/>
 <clearance class="3" value="0.254"/>
 </class>
 <class number="4" name="aref" width="0.254" drill="0.499">
+<clearance class="0" value="0.1524"/>
+<clearance class="1" value="0.1524"/>
+<clearance class="2" value="0.1524"/>
+<clearance class="3" value="0.1524"/>
 <clearance class="4" value="0.254"/>
+</class>
+<class number="5" name="diff pairs" width="0.1524" drill="0">
+<clearance class="0" value="0.1524"/>
+<clearance class="1" value="0.1524"/>
+<clearance class="2" value="0.1524"/>
+<clearance class="3" value="0.1524"/>
+<clearance class="4" value="0.1524"/>
+<clearance class="5" value="0.1524"/>
 </class>
 </classes>
@@
 </segment>
 </net>
-<net name="D-" class="0">
+<net name="D_N" class="5">
 <segment>
 <wire x1="-342.9" y1="-104.14" x2="-347.98" y2="-104.14" width="0.1524" layer="91"/>
@@
 </segment>
 </net>
-<net name="D+" class="0">
+<net name="D_P" class="5">
 <segment>
 <wire x1="-340.36" y1="-106.68" x2="-358.14" y2="-106.68" width="0.1524" layer="91"/>
@@
 </segment>
 </net>
-<net name="RD-" class="0">
-<segment>
-<wire x1="-330.2" y1="-101.6" x2="-320.04" y2="-101.6" width="0.1524" layer="91"/>
-<label x="-320.04" y="-101.6" size="1.778" layer="95" rot="MR0"/>
-<pinref part="R4" gate="G$1" pin="2"/>
-</segment>
-</net>
-<net name="RD+" class="0">
-<segment>
-<wire x1="-330.2" y1="-106.68" x2="-320.04" y2="-106.68" width="0.1524" layer="91"/>
-<label x="-320.04" y="-106.68" size="1.778" layer="95" rot="MR0"/>
-<pinref part="R5" gate="G$1" pin="2"/>
-</segment>
-</net>
-<net name="XUSB" class="3">
+<net name="XUSB" class="0">
 <segment>
 <wire x1="-355.6" y1="-101.6" x2="-355.6" y2="-91.44" width="0.1524" layer="91"/>
@@
 </segment>
 </net>
-<net name="5V" class="0">
+<net name="5V" class="1">
 <segment>
 <wire x1="-309.88" y1="-132.08" x2="-309.88" y2="-129.54" width="0.1524" layer="91"/>
@@
 <pinref part="L3" gate="A" pin="P$1"/>
 <wire x1="-381" y1="-116.84" x2="-378.46" y2="-116.84" width="0.1524" layer="91"/>
+</segment>
+</net>
+<net name="RD_N" class="5">
+<segment>
+<pinref part="R4" gate="G$1" pin="2"/>
+<wire x1="-330.2" y1="-101.6" x2="-320.04" y2="-101.6" width="0.1524" layer="91"/>
+<label x="-327.66" y="-101.6" size="1.778" layer="95"/>
+</segment>
+</net>
+<net name="RD_P" class="5">
+<segment>
+<pinref part="R5" gate="G$1" pin="2"/>
+<wire x1="-330.2" y1="-106.68" x2="-320.04" y2="-106.68" width="0.1524" layer="91"/>
+<label x="-327.66" y="-106.68" size="1.778" layer="95"/>
 </segment>
 </net>
@@
 </segment>
 </net>
-<net name="RD-" class="0">
-<segment>
-<wire x1="116.84" y1="81.28" x2="109.22" y2="81.28" width="0.1524" layer="91"/>
-<label x="106.68" y="81.28" size="1.778" layer="95"/>
-<pinref part="U1" gate="G$1" pin="D-"/>
-</segment>
-</net>
-<net name="RD+" class="0">
-<segment>
-<wire x1="116.84" y1="78.74" x2="109.22" y2="78.74" width="0.1524" layer="91"/>
-<label x="106.68" y="78.74" size="1.778" layer="95"/>
-<pinref part="U1" gate="G$1" pin="D+"/>
-</segment>
-</net>
 <net name="UGND" class="2">
 <segment>
@@
 </segment>
 </net>
-<net name="5V" class="0">
+<net name="5V" class="1">
 <segment>
 <pinref part="U1" gate="G$1" pin="VBUS"/>
@@
 </segment>
 </net>
+<net name="RD_N" class="5">
+<segment>
+<pinref part="U1" gate="G$1" pin="D-"/>
+<wire x1="116.84" y1="81.28" x2="109.22" y2="81.28" width="0.1524" layer="91"/>
+<label x="109.22" y="81.28" size="1.778" layer="95"/>
+</segment>
+</net>
+<net name="RD_P" class="5">
+<segment>
+<pinref part="U1" gate="G$1" pin="D+"/>
+<wire x1="116.84" y1="78.74" x2="109.22" y2="78.74" width="0.1524" layer="91"/>
+<label x="109.22" y="78.74" size="1.778" layer="95"/>
+</segment>
+</net>

Commit message: layout more
Parts:
- added D2, D3: (no value), scono:LED0603
- added J1, J4: i2c, scono:CONN_02
- added J3: spi, scono:CONN_03
- added J5: BURNIN, scono:BURNIN
- added R3, R7: 330R, scono:R-US_0603
Connections:
- new net N$1: D2.C, R3.2
- new net N$2: D3.C, R7.2
- net 5V: now also D2.A, D3.A
- net D0/RX: now also J4.1
- net D1/TX: now also J4.2
- net D2/SDA: now also J1.2
- net D3/SCL: now also J1.1
- net MISO: now also J3.3
- net MOSI: now also J3.2
- net RXLED: now also R7.1
- net SCK: now also J3.1
- net TXLED: now also R3.1

Commit message: finish 32u4 and rev c burnin
Parts:
- added D4: (no value), scono:LED0603
- added J6: GND, scono:CONN_02
- added J7: VCC, scono:CONN_02
- added R8: 330R, scono:R-US_0603
- J4: value i2c -> UART
Connections:
- new net N$4: D4.C, R8.2
- net 5V: now also J5.VCC, J7.1, J7.2
- net D7: now also D4.A
- net GND: now also J5.GND, J6.1, J6.2, R8.1
- net MISO: now also J5.MISO
- net MOSI: now also J5.MOSI
- net RESET: now also J5.RST
- net SCK: now also J5.SCK
Changed lines of the file:
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@@
 <?xml version="1.0" encoding="utf-8"?>
 <!DOCTYPE eagle SYSTEM "eagle.dtd">
-<eagle version="9.5.0">
+<eagle version="9.5.1">
 <drawing>
 <settings>
@@
 <part name="U$1" library="scono" library_urn="urn:adsk.eagle:library:14850048" deviceset="5V" device=""/>
 <part name="U$2" library="scono" library_urn="urn:adsk.eagle:library:14850048" deviceset="5V" device=""/>
-<part name="J4" library="scono" library_urn="urn:adsk.eagle:library:14850048" deviceset="CONN_02" device="" package3d_urn="urn:adsk.eagle:package:38039/1" value="i2c"/>
+<part name="J4" library="scono" library_urn="urn:adsk.eagle:library:14850048" deviceset="CONN_02" device="" package3d_urn="urn:adsk.eagle:package:38039/1" value="UART"/>
 <part name="J5" library="scono" library_urn="urn:adsk.eagle:library:14850048" deviceset="BURNIN" device="" package3d_urn="urn:adsk.eagle:package:14850856/1"/>
+<part name="U$9" library="scono" library_urn="urn:adsk.eagle:library:14850048" deviceset="5V" device=""/>
+<part name="SUPPLY3" library="scono" library_urn="urn:adsk.eagle:library:14850048" deviceset="GND" device=""/>
+<part name="J6" library="scono" library_urn="urn:adsk.eagle:library:14850048" deviceset="CONN_02" device="" package3d_urn="urn:adsk.eagle:package:38039/1" value="GND"/>
+<part name="J7" library="scono" library_urn="urn:adsk.eagle:library:14850048" deviceset="CONN_02" device="" package3d_urn="urn:adsk.eagle:package:38039/1" value="VCC"/>
+<part name="SUPPLY4" library="scono" library_urn="urn:adsk.eagle:library:14850048" deviceset="GND" device=""/>
+<part name="U$10" library="scono" library_urn="urn:adsk.eagle:library:14850048" deviceset="5V" device=""/>
+<part name="R8" library="scono" library_urn="urn:adsk.eagle:library:14850048" deviceset="R-US_" device="0603" package3d_urn="urn:adsk.eagle:package:14850803/1" value="330R"/>
+<part name="D4" library="scono" library_urn="urn:adsk.eagle:library:14850048" deviceset="LED" device="0603" package3d_urn="urn:adsk.eagle:package:14850721/1"/>
+<part name="SUPPLY17" library="scono" library_urn="urn:adsk.eagle:library:14850048" deviceset="GND" device=""/>
 </parts>
 <sheets>
@@
 <attribute name="NAME" x="55.88" y="172.72" size="1.778" layer="94" align="top-left"/>
 </instance>
+<instance part="U$9" gate="G$1" x="48.26" y="167.64" smashed="yes" rot="R90">
+<attribute name="VALUE" x="44.45" y="166.37" size="1.778" layer="96" rot="R90"/>
+</instance>
+<instance part="SUPPLY3" gate="GND" x="48.26" y="152.4" smashed="yes">
+<attribute name="VALUE" x="46.99" y="149.86" size="1.016" layer="96"/>
+</instance>
+<instance part="J6" gate="G$1" x="60.96" y="33.02" smashed="yes">
+<attribute name="VALUE" x="58.42" y="28.194" size="1.778" layer="96" font="vector"/>
+<attribute name="NAME" x="58.42" y="38.608" size="1.778" layer="95" font="vector"/>
+</instance>
+<instance part="J7" gate="G$1" x="60.96" y="17.78" smashed="yes">
+<attribute name="VALUE" x="58.42" y="12.954" size="1.778" layer="96" font="vector"/>
+<attribute name="NAME" x="58.42" y="23.368" size="1.778" layer="95" font="vector"/>
+</instance>
+<instance part="SUPPLY4" gate="GND" x="71.12" y="35.56" smashed="yes" rot="R90">
+<attribute name="VALUE" x="73.66" y="34.29" size="1.016" layer="96" rot="R90"/>
+</instance>
+<instance part="U$10" gate="G$1" x="68.58" y="20.32" smashed="yes" rot="R270">
+<attribute name="VALUE" x="72.39" y="21.59" size="1.778" layer="96" rot="R270"/>
+</instance>
+<instance part="R8" gate="G$1" x="223.52" y="45.72" smashed="yes" rot="R180">
+<attribute name="NAME" x="228.6" y="44.45" size="1.016" layer="95" rot="R180"/>
+<attribute name="VALUE" x="228.6" y="46.99" size="1.016" layer="96" rot="R180" align="top-left"/>
+</instance>
+<instance part="D4" gate="G$1" x="215.9" y="45.72" smashed="yes" rot="R90">
+<attribute name="NAME" x="220.472" y="42.291" size="1.778" layer="95" font="vector" rot="R180"/>
+<attribute name="VALUE" x="220.472" y="47.625" size="1.778" layer="96" font="vector" rot="R180" align="top-left"/>
+</instance>
+<instance part="SUPPLY17" gate="GND" x="231.14" y="45.72" smashed="yes" rot="R90">
+<attribute name="VALUE" x="233.68" y="44.45" size="1.016" layer="96" rot="R90"/>
+</instance>
 </instances>
 <busses>
@@
 <pinref part="SUPPLY15" gate="GND" pin="GND"/>
 </segment>
+<segment>
+<pinref part="J5" gate="G$1" pin="GND"/>
+<wire x1="53.34" y1="154.94" x2="48.26" y2="154.94" width="0.1524" layer="91"/>
+<pinref part="SUPPLY3" gate="GND" pin="GND"/>
+</segment>
+<segment>
+<pinref part="J6" gate="G$1" pin="2"/>
+<pinref part="SUPPLY4" gate="GND" pin="GND"/>
+<pinref part="J6" gate="G$1" pin="1"/>
+<wire x1="68.58" y1="35.56" x2="68.58" y2="33.02" width="0.1524" layer="91"/>
+<junction x="68.58" y="35.56"/>
+</segment>
+<segment>
+<pinref part="R8" gate="G$1" pin="1"/>
+<pinref part="SUPPLY17" gate="GND" pin="GND"/>
+</segment>
 </net>
 <net name="AREF" class="4">
@@
 <pinref part="SW1" gate="G$1" pin="B"/>
 </segment>
+<segment>
+<pinref part="J5" gate="G$1" pin="RST"/>
+<wire x1="53.34" y1="157.48" x2="48.26" y2="157.48" width="0.1524" layer="91"/>
+<label x="48.26" y="157.48" size="1.778" layer="95" rot="R180"/>
+</segment>
 </net>
 <net name="SCK" class="0">
@@
 <pinref part="J3" gate="J$1" pin="1"/>
 </segment>
+<segment>
+<pinref part="J5" gate="G$1" pin="SCK"/>
+<wire x1="53.34" y1="165.1" x2="48.26" y2="165.1" width="0.1524" layer="91"/>
+<label x="48.26" y="165.1" size="1.778" layer="95" rot="R180"/>
+</segment>
 </net>
 <net name="MISO" class="0">
@@
 <pinref part="J3" gate="J$1" pin="3"/>
 </segment>
+<segment>
+<pinref part="J5" gate="G$1" pin="MISO"/>
+<wire x1="53.34" y1="162.56" x2="48.26" y2="162.56" width="0.1524" layer="91"/>
+<label x="48.26" y="162.56" size="1.778" layer="95" rot="R180"/>
+</segment>
 </net>
 <net name="MOSI" class="0">
@@
 <label x="43.18" y="53.34" size="1.778" layer="95"/>
 <pinref part="J3" gate="J$1" pin="2"/>
+</segment>
+<segment>
+<pinref part="J5" gate="G$1" pin="MOSI"/>
+<wire x1="53.34" y1="160.02" x2="48.26" y2="160.02" width="0.1524" layer="91"/>
+<label x="48.26" y="160.02" size="1.778" layer="95" rot="R180"/>
 </segment>
 </net>
@@
 <pinref part="U$2" gate="G$1" pin="5V"/>
 </segment>
+<segment>
+<pinref part="J5" gate="G$1" pin="VCC"/>
+<wire x1="53.34" y1="167.64" x2="48.26" y2="167.64" width="0.1524" layer="91"/>
+<pinref part="U$9" gate="G$1" pin="5V"/>
+</segment>
+<segment>
+<pinref part="J7" gate="G$1" pin="2"/>
+<pinref part="U$10" gate="G$1" pin="5V"/>
+<pinref part="J7" gate="G$1" pin="1"/>
+<wire x1="68.58" y1="20.32" x2="68.58" y2="17.78" width="0.1524" layer="91"/>
+<junction x="68.58" y="20.32"/>
+</segment>
 </net>
 <net name="AGND" class="0">
@@
 <pinref part="U1" gate="G$1" pin="(INT6/AIN0)PE6"/>
 </segment>
+<segment>
+<pinref part="D4" gate="G$1" pin="A"/>
+<wire x1="213.36" y1="45.72" x2="210.82" y2="45.72" width="0.1524" layer="91"/>
+<label x="208.28" y="45.72" size="1.778" layer="95"/>
+</segment>
 </net>
 <net name="UCAP" class="0">
@@
 </segment>
 </net>
+<net name="N$4" class="0">
+<segment>
+<pinref part="R8" gate="G$1" pin="2"/>
+<pinref part="D4" gate="G$1" pin="C"/>
+</segment>
+</net>

Commit message: Add same pinpouts as mipp_v2
Parts:
- removed J1: i2c, scono:CONN_02
- removed J3: spi, scono:CONN_03
- removed J4: UART, scono:CONN_02
- removed J6: GND, scono:CONN_02
- removed J7: VCC, scono:CONN_02
- added U2: MIPPE, scono:MIPPE
Connections:
- net 5V: now also U2.VCC; no longer J7.1, J7.2
- net A0: now also U2.ADC0
- net A1: now also U2.ADC1
- net A2: now also U2.ADC2
- net A3: now also U2.ADC3
- net D0/RX: now also U2.RX; no longer J4.1
- net D1/TX: now also U2.TX; no longer J4.2
- net D2/SDA: now also U2.SDA; no longer J1.2
- net D3/SCL: now also U2.SCL; no longer J1.1
- net D4: now also U2.SS
- net GND: now also U2.GND; no longer J6.1, J6.2
- net IO10*: now also U2.GPIO5
- net IO11*: now also U2.GPIO6
- net IO8: now also U2.GPIO3
- net IO9*: now also U2.GPIO4
- net MISO: now also U2.MISO; no longer J3.3
- net MOSI: now also U2.MOSI; no longer J3.2
- net SCK: now also U2.SCK; no longer J3.1
