File: oled_pmic/oled_pmic.brd (EAGLE design)
At the start: 160 x 100 mm, 11 parts, among them J1 I_sense, J2 VCC, J4 GND, Q1 N-CHANNEL-MOSFETSOT23-3, U1 AL5801W6-7

Commit message: layout board
Parts:
- moved J4 44.9 mm to (12.0, 4.00), turned to 270 degrees
- moved J3 43.3 mm to (12.0, 7.00), turned to 90 degrees
- moved J2 39.5 mm to (3.50, 12.0), turned to 180 degrees
- moved Q1 37.2 mm to (7.00, 12.0), turned to 180 degrees
- moved U1 29.7 mm to (8.00, 4.50)
- moved R1 28.4 mm to (8.07, 8.63), turned to 180 degrees
- moved D2 27.0 mm to (7.00, 0.75)
- moved D1 24.5 mm to (2.25, 0.75)
- moved J1 21.3 mm to (3.50, 3.50), turned to 180 degrees
- moved R2 19.1 mm to (3.50, 8.00), turned to 90 degrees
- moved C1 15.5 mm to (0.25, 8.00), turned to 90 degrees
Routing:
- net BIAS: track 0.00 -> 14.9 mm
- net FB: track 0.00 -> 14.3 mm, vias 0 -> 2
- net GND: track 0.00 -> 5.94 mm, vias 0 -> 3
- net PWM: track 0.00 -> 4.43 mm
- net N$3: track 0.00 -> 3.32 mm
- net N$2: track 0.00 -> 3.00 mm
- net N$4: track 0.00 -> 2.92 mm
- added copper zone on layer 16, net GND
- added copper zone on layer 1, net VCC
Other:
- board size 160 x 100 mm -> 16.5 x 16 mm
- board text added: "BIAS"
- board text added: "FB"
- board text added: "GND"
- board text added: "PWM"
- board text added: "VCC"

Commit message: place order
Parts:
- moved C1 1.80 mm to (1.75, 9.00)
- moved D1 1.80 mm to (3.75, 1.75)
- moved D2 1.80 mm to (8.50, 1.75)
- moved J1 1.80 mm to (5.00, 4.50)
- moved J2 1.80 mm to (5.00, 13.0)
- moved J3 1.80 mm to (13.5, 8.00)
- moved J4 1.80 mm to (13.5, 5.00)
- moved Q1 1.80 mm to (8.50, 13.0)
- moved R1 1.80 mm to (9.57, 9.63)
- moved R2 1.80 mm to (5.00, 9.00)
- moved U1 1.80 mm to (9.50, 5.50)
