File: mippe_mobo/mippe_mobo.sch (EAGLE design)
At the start: 43 parts, among them J3 FFC-32, J5 BURNIN, SW1 BTN-PTS810, U1 CD4052BPWR, U2 LM340MPX-5.0230, U3 ATMEGA32U4-XUAU, X1 USB-B1HSB6, Y1 16MHz

Commit message: more mobo work
Parts:
- removed C8: 0.1uF, scono:CAP0402-CAP
- removed D1: (no value), scono:LED0603
- removed R13: 330R, scono:R-US_R0402
- removed U2: LM340MPX-5.0230, scono:LM340MPX-5.0230
Connections:
- removed net D7: D1.A
- removed net N$35: D1.C, R13.2
- net 5V: now also R1.1, R2.1, R3.1, R4.1, R5.1, R6.1; no longer C8.2, U2.5V
- net GND: now also C1.1; no longer C8.1, R13.1, U2.GND
- net VCC: no longer R1.1, R2.1, R3.1, R4.1, R5.1, R6.1, U2.VIN

Commit message: mobo work
Parts:
- added J4: PJ-102AH, scono:PJ-102AH
- added L1: UCB_CAL500MIL, scono:UCB_CAL500MIL
Connections:
- net GND: now also J4.1, J4.3
- net VCC: now also J4.2

Commit message: more progress add ss
Parts:
- added J6, J7: (no value), scono:CONN_04
Connections:
- net GND: now also J6.1, J6.2, J6.3, J6.4, J7.1, J7.2, J7.3, J7.4
Changed lines of the file:
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@@
 <part name="SUPPLY7" library="scono" library_urn="urn:adsk.eagle:library:14850048" deviceset="GND" device=""/>
 <part name="SUPPLY8" library="scono" library_urn="urn:adsk.eagle:library:14850048" deviceset="VCC" device=""/>
+<part name="J6" library="scono" library_urn="urn:adsk.eagle:library:14850048" deviceset="CONN_04" device="" package3d_urn="urn:adsk.eagle:package:38085/1"/>
+<part name="SUPPLY9" library="scono" library_urn="urn:adsk.eagle:library:14850048" deviceset="GND" device=""/>
+<part name="J7" library="scono" library_urn="urn:adsk.eagle:library:14850048" deviceset="CONN_04" device="" package3d_urn="urn:adsk.eagle:package:38085/1"/>
+<part name="SUPPLY10" library="scono" library_urn="urn:adsk.eagle:library:14850048" deviceset="GND" device=""/>
 </parts>
 <sheets>
@@
 <attribute name="VALUE" x="60.94716875" y="60.8787" size="1.780990625" layer="96"/>
 </instance>
+<instance part="J6" gate="G$1" x="116.84" y="154.94" smashed="yes">
+<attribute name="VALUE" x="111.76" y="147.574" size="1.778" layer="96" font="vector"/>
+<attribute name="NAME" x="111.76" y="163.068" size="1.778" layer="95" font="vector"/>
+</instance>
+<instance part="SUPPLY9" gate="GND" x="121.92" y="149.86" smashed="yes"/>
+<instance part="J7" gate="G$1" x="116.84" y="137.16" smashed="yes">
+<attribute name="VALUE" x="111.76" y="129.794" size="1.778" layer="96" font="vector"/>
+<attribute name="NAME" x="111.76" y="145.288" size="1.778" layer="95" font="vector"/>
+</instance>
+<instance part="SUPPLY10" gate="GND" x="121.92" y="132.08" smashed="yes"/>
 </instances>
 <busses>
@@
 </segment>
 </net>
+<net name="GND" class="0">
+<segment>
+<pinref part="J6" gate="G$1" pin="1"/>
+<pinref part="SUPPLY9" gate="GND" pin="GND"/>
+<pinref part="J6" gate="G$1" pin="2"/>
+<wire x1="121.92" y1="152.4" x2="121.92" y2="154.94" width="0.1524" layer="91"/>
+<junction x="121.92" y="152.4"/>
+<pinref part="J6" gate="G$1" pin="3"/>
+<wire x1="121.92" y1="154.94" x2="121.92" y2="157.48" width="0.1524" layer="91"/>
+<junction x="121.92" y="154.94"/>
+<pinref part="J6" gate="G$1" pin="4"/>
+<wire x1="121.92" y1="157.48" x2="121.92" y2="160.02" width="0.1524" layer="91"/>
+<junction x="121.92" y="157.48"/>
+</segment>
+<segment>
+<pinref part="J7" gate="G$1" pin="1"/>
+<pinref part="SUPPLY10" gate="GND" pin="GND"/>
+<pinref part="J7" gate="G$1" pin="2"/>
+<wire x1="121.92" y1="134.62" x2="121.92" y2="137.16" width="0.1524" layer="91"/>
+<junction x="121.92" y="134.62"/>
+<pinref part="J7" gate="G$1" pin="3"/>
+<wire x1="121.92" y1="137.16" x2="121.92" y2="139.7" width="0.1524" layer="91"/>
+<junction x="121.92" y="137.16"/>
+<pinref part="J7" gate="G$1" pin="4"/>
+<wire x1="121.92" y1="139.7" x2="121.92" y2="142.24" width="0.1524" layer="91"/>
+<junction x="121.92" y="139.7"/>
+</segment>
+</net>
