File: mippe_mobo/mippe_mobo.brd (EAGLE design)
At the start: 160 x 120 mm, 43 parts, among them J3 FFC-32, J5 BURNIN, SW1 BTN-PTS810, U1 CD4052BPWR, U2 LM340MPX-5.0230, U3 ATMEGA32U4-XUAU, X1 USB-B1HSB6, Y1 16MHz

Commit message: more mobo work
Parts:
- removed C8: 0.1uF, scono:0402-CAP
- removed D1: (no value), scono:LED-0603
- removed R13: 330R, scono:R0402
- removed U2: LM340MPX-5.0230, scono:SOT230P700X180-4N
- moved R2 183.5 mm to (14.5, 96.8), turned to 90 degrees
- moved R3 178.0 mm to (5.00, 96.8), turned to 90 degrees
- moved C1 173.2 mm to (9.75, 102.8)
- moved R1 172.3 mm to (5.00, 102.8), turned to 270 degrees
- moved U1 165.7 mm to (9.75, 99.0)
- moved R6 117.5 mm to (14.5, 99.8), turned to 90 degrees
- moved R4 109.8 mm to (14.5, 102.8), turned to 270 degrees
- moved R5 104.2 mm to (5.00, 99.8), turned to 90 degrees
- moved C9 42.9 mm to (29.0, 97.5), turned to 270 degrees
- moved D3 42.3 mm to (13.8, 117.5), turned to 90 degrees
- moved R12 41.7 mm to (12.5, 117.5), turned to 90 degrees
- moved SW1 39.3 mm to (36.2, 117.2)
- moved Y1 39.3 mm to (24.5, 97.5), turned to 180 degrees
- moved R10 39.3 mm to (32.2, 116.8)
- moved R11 37.6 mm to (11.2, 117.5), turned to 90 degrees
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Connections:
- removed net D7: D1.A
- removed net N$35: D1.C, R13.2
- net 5V: now also R1.1, R2.1, R3.1, R4.1, R5.1, R6.1; no longer C8.2, U2.3
- net GND: now also C1.1; no longer C8.1, R13.1, U2.2, U2.4
- net VCC: no longer R1.1, R2.1, R3.1, R4.1, R5.1, R6.1, U2.1
Routing:
- net GND: track 0.20 -> 227.0 mm, vias 0 -> 19
- net VCC: track 0.00 -> 200.9 mm, vias 0 -> 1
- net RESET: track 0.00 -> 36.0 mm, vias 0 -> 2
- net TXLED: track 0.00 -> 28.6 mm, vias 0 -> 2
- net TX: track 0.00 -> 23.9 mm, vias 0 -> 2
- net MISO: track 0.00 -> 21.0 mm, vias 0 -> 1
- net RX: track 0.00 -> 20.1 mm, vias 0 -> 2
- net RXLED: track 0.00 -> 19.3 mm, vias 0 -> 2
- net SCK: track 0.00 -> 18.7 mm, vias 0 -> 1
- net TX2: track 0.00 -> 18.5 mm, vias 0 -> 1
- net MOSI: track 0.00 -> 17.1 mm, vias 0 -> 1
- net RX3: track 0.00 -> 12.8 mm, vias 0 -> 1
- net RX1: track 0.00 -> 12.7 mm, vias 0 -> 2
- net D_P: track 0.00 -> 11.9 mm
- net D_N: track 0.00 -> 11.7 mm
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- added copper zone on layer 1, net 5V
- added copper zone on layer 16, net GND
Other:
- board size 160 x 120 mm -> 120 x 120 mm
- board text added: "TX RX"

Commit message: mobo work
Parts:
- added J4: PJ-102AH, scono:CUI_PJ-102AH
- added L1: UCB_CAL500MIL, scono:UCB_CAL_500MIL
- added U$17: (no value), pie:OSHW-LOGO-L
Connections:
- net GND: now also J4.1, J4.3
- net VCC: now also J4.2
Routing:
- net RX2: track 6.33 -> 62.8 mm
- net TX2: track 18.5 -> 70.1 mm, vias 1 -> 2
- net TX3: track 7.65 -> 56.9 mm, vias 0 -> 2
- net VCC: track 200.9 -> 248.6 mm
- net RX3: track 12.8 -> 60.4 mm, vias 1 -> 2
- net GND: track 227.0 -> 266.7 mm, vias 19 -> 21
- net TX1: track 7.69 -> 27.6 mm
- net RX1: track 12.7 -> 31.2 mm
Other:
- board text added: "Modular Integration Platform for Printed Electronics Arias Research Group Design: Seiya Ono '20 https://github.com/onibrow/arg-mippe/wiki"

Commit message: more progress add ss
Parts:
- added J6, J7: (no value), scono:1X04
- moved J1 1.25 mm to (-39.2, 14.2)
- moved J2 1.25 mm to (-39.2, 11.8)
Connections:
- net GND: now also J6.1, J6.2, J6.3, J6.4, J7.1, J7.2, J7.3, J7.4
Routing:
- net GND: track 266.7 -> 325.1 mm
- net N$20: track 12.9 -> 14.1 mm
- net N$19: track 10.9 -> 12.2 mm
- net N$18: track 10.1 -> 11.4 mm
- net N$17: track 9.35 -> 10.6 mm
- net N$16: track 9.20 -> 10.4 mm
- net N$15: track 10.0 -> 11.3 mm
- net N$14: track 10.8 -> 12.0 mm
- net N$5: track 28.7 -> 29.3 mm
- net N$9: track 20.6 -> 21.1 mm
- net N$8: track 22.6 -> 23.1 mm
- net N$7: track 24.6 -> 25.1 mm
- net N$4: track 30.9 -> 31.4 mm
- net N$32: track 36.8 -> 37.3 mm
- net N$31: track 35.1 -> 35.6 mm
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Other:
- board text added: "1"
- board text added: "10"
- board text added: "11"
- board text added: "12"
- board text added: "13"
- board text added: "14"
- board text added: "15"
- board text added: "16"
- board text added: "17"
- board text added: "18"
- board text added: "19"
- board text added: "2"
- board text added: "20"
- board text added: "21"
- board text added: "22"
- board text added: "23"
- board text added: "24"
- board text added: "25"
- board text added: "26"
- board text added: "27"
- board text added: "28"
- board text added: "29"
- board text added: "3"
- board text added: "30"
- board text added: "31"
- board text added: "32"
- board text added: "4"
- board text added: "5"
- board text added: "6"
- board text added: "7"
- board text added: "8"
- board text added: "9"
- board text added: "GND"
- board text added: "Module 1"
- board text added: "Module 2"
- board text added: "Module 3"

Commit message: finalize mobo
Parts:
- added C8: (no value), scono:CAP_3MM
- added D1: (no value), scono:LED-0603
- added R13, R14: 10k, scono:R0402
- added R15: 330R, scono:R0402
- added TP1, TP2, TP3, TP4, TP5: TEST_POINTTHRU, scono:TEST_POINT
- U3: value ATMEGA32U4-XUAU -> ATMEGA32U4-XUMU; device scono:TQFP44-PAD -> scono:QFN44ML7X7
- moved C7 60.2 mm to (75.5, 105.5)
- moved R4 60.1 mm to (74.5, 99.8), turned to 90 degrees
- moved R6 60.1 mm to (74.5, 102.8), turned to 270 degrees
- moved B1 60.0 mm to (60.0, 40.0)
- moved B2 60.0 mm to (20.0, 25.0)
- moved B3 60.0 mm to (100.0, 25.0)
- moved C1 60.0 mm to (69.8, 102.8)
- moved C10 60.0 mm to (80.0, 97.2)
- moved C2 60.0 mm to (90.8, 112.0)
- moved C3 60.0 mm to (78.8, 116.8)
- moved C4 60.0 mm to (90.8, 100.8)
- moved C5 60.0 mm to (79.2, 112.0)
- moved C6 60.0 mm to (79.2, 100.8)
- moved C9 60.0 mm to (89.0, 97.5)
- moved D2 60.0 mm to (70.0, 117.5)
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Connections:
- new net N$35: D1.C, R15.2
- net 5V: now also D1.A, R13.2, R14.2, TP5.1
- net A: now also U3.18
- net B: now also U3.19
- net GND: now also C8.NEG, R15.1, TP3.1, U3.EXP; no longer U3.P$1
- net RX4: now also R14.1, TP1.1
- net TX2: now also U1.14; no longer U1.15
- net TX3: now also U1.15; no longer U1.14
- net TX4: now also R13.1, TP2.1
- net VCC: now also C8.POS, TP4.1
Routing:
- net B: track 0.00 -> 23.1 mm, vias 0 -> 2
- net A: track 0.00 -> 21.7 mm, vias 0 -> 2
- net GND: track 325.1 -> 346.8 mm, vias 21 -> 28
- net RX4: track 0.00 -> 15.0 mm, vias 0 -> 1
- net TX4: track 0.00 -> 14.9 mm, vias 0 -> 1
- net VCC: track 248.6 -> 262.5 mm, vias 1 -> 2
- net RXLED: track 19.3 -> 24.2 mm, vias 2 -> 3
- net RESET: track 36.0 -> 40.3 mm, vias 2 -> 5
- net AREF: track 7.92 -> 11.8 mm, vias 0 -> 2
- net AGND: track 6.76 -> 10.4 mm, vias 0 -> 2
- net HWB: track 2.37 -> 5.24 mm
- net RD_N: track 7.37 -> 10.2 mm
- net XTAL2: track 6.69 -> 9.34 mm
- net RD_P: track 7.17 -> 9.80 mm
- net XTAL1: track 6.50 -> 9.03 mm
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Other:
- board text added: "5V"

Commit message: add more ground pins to mobo
Parts:
- added J10, J11, J8, J9: (no value), scono:1X04
Connections:
- net GND: now also J10.1, J10.2, J10.3, J10.4, J11.1, J11.2, J11.3, J11.4, J8.1, J8.2, J8.3, J8.4, J9.1, J9.2, J9.3, J9.4
Routing:
- net GND: track 346.8 -> 437.3 mm
Changed lines of the file:
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@@
 <attribute name="VALUE" x="91.98" y="103.143" size="0.508" layer="27" font="vector" rot="R270"/>
+</element>
+<element name="J8" library="scono" library_urn="urn:adsk.eagle:library:14850048" package="1X04" package3d_urn="urn:adsk.eagle:package:38085/1" value="" x="15" y="15" smashed="yes" rot="R180">
+<attribute name="PROD_ID" value="CONN-09696" x="15" y="15" size="1.778" layer="27" rot="R180" display="off"/>
+<attribute name="VALUE" x="16.27" y="17.032" size="0.6096" layer="27" font="vector" ratio="20" rot="R180"/>
+</element>
+<element name="J9" library="scono" library_urn="urn:adsk.eagle:library:14850048" package="1X04" package3d_urn="urn:adsk.eagle:package:38085/1" value="" x="15" y="17.75" smashed="yes" rot="R180">
+<attribute name="PROD_ID" value="CONN-09696" x="15" y="17.75" size="1.778" layer="27" rot="R180" display="off"/>
+<attribute name="VALUE" x="16.27" y="19.782" size="0.6096" layer="27" font="vector" ratio="20" rot="R180"/>
+</element>
+<element name="J10" library="scono" library_urn="urn:adsk.eagle:library:14850048" package="1X04" package3d_urn="urn:adsk.eagle:package:38085/1" value="" x="105" y="17.75" smashed="yes">
+<attribute name="PROD_ID" value="CONN-09696" x="105" y="17.75" size="1.778" layer="27" display="off"/>
+<attribute name="VALUE" x="103.73" y="15.718" size="0.6096" layer="27" font="vector" ratio="20"/>
+</element>
+<element name="J11" library="scono" library_urn="urn:adsk.eagle:library:14850048" package="1X04" package3d_urn="urn:adsk.eagle:package:38085/1" value="" x="105" y="15" smashed="yes">
+<attribute name="PROD_ID" value="CONN-09696" x="105" y="15" size="1.778" layer="27" display="off"/>
+<attribute name="VALUE" x="103.73" y="12.968" size="0.6096" layer="27" font="vector" ratio="20"/>
 </element>
 </elements>
@@
 <via x="93.25" y="102.65" extent="1-16" drill="0.2"/>
 <via x="74.85" y="105.5" extent="1-16" drill="0.2"/>
+<contactref element="J8" pad="1"/>
+<contactref element="J8" pad="2"/>
+<contactref element="J8" pad="3"/>
+<contactref element="J8" pad="4"/>
+<contactref element="J9" pad="1"/>
+<contactref element="J9" pad="2"/>
+<contactref element="J9" pad="3"/>
+<contactref element="J9" pad="4"/>
+<contactref element="J10" pad="1"/>
+<contactref element="J10" pad="2"/>
+<contactref element="J10" pad="3"/>
+<contactref element="J10" pad="4"/>
+<contactref element="J11" pad="1"/>
+<contactref element="J11" pad="2"/>
+<contactref element="J11" pad="3"/>
+<contactref element="J11" pad="4"/>
+<wire x1="87.546" y1="27.204" x2="97" y2="17.75" width="1" layer="16"/>
+<wire x1="97" y1="17.75" x2="105" y2="17.75" width="1" layer="16"/>
+<wire x1="7.546" y1="27.204" x2="7.546" y2="17.916" width="1" layer="16"/>
+<wire x1="7.546" y1="17.916" x2="7.38" y2="17.75" width="1" layer="16"/>
+<wire x1="7.38" y1="17.75" x2="9.92" y2="17.75" width="1" layer="16"/>
+<wire x1="9.92" y1="17.75" x2="12.46" y2="17.75" width="1" layer="16"/>
+<wire x1="12.46" y1="17.75" x2="15" y2="17.75" width="1" layer="16"/>
+<wire x1="15" y1="17.75" x2="15" y2="15" width="1" layer="16"/>
+<wire x1="15" y1="15" x2="12.46" y2="15" width="1" layer="16"/>
+<wire x1="12.46" y1="15" x2="9.92" y2="15" width="1" layer="16"/>
+<wire x1="9.92" y1="15" x2="7.38" y2="15" width="1" layer="16"/>
+<wire x1="7.38" y1="15" x2="7.38" y2="17.75" width="1" layer="16"/>
+<wire x1="9.92" y1="17.75" x2="9.92" y2="15" width="1" layer="16"/>
+<wire x1="12.46" y1="17.75" x2="12.46" y2="15" width="1" layer="16"/>
+<wire x1="105" y1="17.75" x2="105" y2="15" width="1" layer="16"/>
+<wire x1="107.54" y1="17.75" x2="107.54" y2="15" width="1" layer="16"/>
+<wire x1="110.08" y1="17.75" x2="110.08" y2="15" width="1" layer="16"/>
+<wire x1="112.62" y1="17.75" x2="112.62" y2="15" width="1" layer="16"/>
+<wire x1="105" y1="15" x2="107.54" y2="15" width="1" layer="16"/>
+<wire x1="107.54" y1="15" x2="110.08" y2="15" width="1" layer="16"/>
+<wire x1="110.08" y1="15" x2="112.62" y2="15" width="1" layer="16"/>
+<wire x1="112.62" y1="17.75" x2="110.08" y2="17.75" width="1" layer="16"/>
+<wire x1="110.08" y1="17.75" x2="107.54" y2="17.75" width="1" layer="16"/>
+<wire x1="107.54" y1="17.75" x2="105" y2="17.75" width="1" layer="16"/>
+<wire x1="56.25" y1="29" x2="58.25" y2="29" width="1" layer="16"/>
+<wire x1="61.33" y1="29" x2="58.79" y2="29" width="1" layer="16"/>
+<wire x1="61.33" y1="29" x2="63.87" y2="29" width="1" layer="16"/>
 </signal>
 <signal name="TX1">
@@
 </polygon>
 <contactref element="TP5" pad="1"/>
-<contactref element="TP5" pad="1"/>
 <wire x1="95.75" y1="113.75" x2="93.25" y2="113.75" width="0.5" layer="16"/>

Commit message: finish boms and cams
Parts:
- moved L1 89.2 mm to (12.2, 78.2)
- moved U$17 8.70 mm to (107.8, 106.0)
Changed lines of the file:
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@@
 <attribute name="VALUE" x="50.638490625" y="122.5129" size="1.271559375" layer="27" rot="R270"/>
 </element>
-<element name="L1" library="scono" library_urn="urn:adsk.eagle:library:14850048" package="UCB_CAL_500MIL" value="UCB_CAL500MIL" x="99.75" y="95.75" smashed="yes"/>
+<element name="L1" library="scono" library_urn="urn:adsk.eagle:library:14850048" package="UCB_CAL_500MIL" value="UCB_CAL500MIL" x="12.25" y="78.25" smashed="yes"/>
 <element name="J4" library="scono" library_urn="urn:adsk.eagle:library:14850048" package="CUI_PJ-102AH" value="PJ-102AH" x="44" y="115" smashed="yes" rot="R90">
 <attribute name="AVAILABILITY" value="Unavailable" x="44" y="115" size="1.778" layer="27" rot="R90" display="off"/>
@@
 <attribute name="VALUE" x="50.41615" y="107.8031" size="1.27121875" layer="27" rot="R90"/>
 </element>
-<element name="U$17" library="pie" package="OSHW-LOGO-L" value="" x="110.5" y="114.25" smashed="yes"/>
+<element name="U$17" library="pie" package="OSHW-LOGO-L" value="" x="107.75" y="106" smashed="yes"/>
 <element name="J6" library="scono" library_urn="urn:adsk.eagle:library:14850048" package="1X04" package3d_urn="urn:adsk.eagle:package:38085/1" value="" x="56.25" y="26.25" smashed="yes">
 <attribute name="PROD_ID" value="CONN-09696" x="56.25" y="26.25" size="1.778" layer="27" display="off"/>
