File: act_pot_diff/act_pot_diff.sch (EAGLE design)
At the start: 11 parts, among them J1 FFC-32, J2 REF_GND, J3 SENSORS, J4 I2C, J5 GND, J6 VDD, U1 MCP3424T-E/ST, U2 LM340MPX-5.0230

Commit message: finish module and diff module
Parts:
- added C10, C11, C12, C14, C15, C16, C17, C7, C9: 0.1uF, scono:CAP0402-CAP
- added C13, C8: 0.1uF, scono:CAP0603-CAP
- added C2, C3, C4: 100nF, scono:CAP0402-CAP
- added C5, C6: 18pF, scono:CAP0402-CAP
- added D1: (no value), scono:LED0603
- added D2: RED, scono:LED0603
- added J10: I2C, scono:CONN_02
- added J12: BURNIN, scono:BURNIN
- added J9: (no value), scono:CONN_08"
- added R1, R4, R5: 10k, scono:R-US_R0402
- added SW1: BTN-PTS810, scono:BTN-PTS810
- added TP1: TEST_POINTTHRU, scono:TEST_POINTTHRU
- added U3, U4: MCP3424T-E/ST, scono:MCP3424T-E/ST
- added Y1: 16MHz, scono:CRYSTAL_SMOL
- C1: value (none) -> 100nF; device scono:CAP0603-CAP -> scono:CAP0402-CAP
- J1: value FFC-32 -> VCC; device scono:FFC-32 -> scono:CONN_02
- J2: value REF_GND -> GND
- J3: value SENSORS -> UART; device scono:CONN_04 -> scono:CONN_02
- J4: value I2C -> FTDI; device scono:CONN_02 -> scono:CONN_06NO_SILK_FEMALE_PTH
- J5: value GND -> VCC
- J6: value VDD -> GND
- R2, R3: value 10k -> 500R; device scono:R-US_0603 -> scono:R-US_R0402
- U1: value MCP3424T-E/ST -> LM340MPX-5.0230; device scono:MCP3424T-E/ST -> scono:LM340MPX-5.0230
- U2: value LM340MPX-5.0230 -> ATMEGA328P-AUR; device scono:LM340MPX-5.0230 -> scono:ATMEGA328P-AUR
Connections:
- removed net K: J1.18, J1.19, J1.20, J1.21, J1.22, J3.3, U1.CH3+
- removed net NA: J1.11, J1.12, J1.13, J1.14, J1.15, J3.2, U1.CH2+
- removed net NH4: J1.4, J1.5, J1.6, J1.7, J1.8, J3.1, U1.CH1+
- removed net REF_ELEC: J1.25, J1.26, J1.27, J1.28, J1.29, J2.1, J3.4, U1.CH1-, U1.CH2-, U1.CH3-
- new net ADC0: U2.PC0(ADC0/PCINT8)
- new net ADC1: U2.PC1(ADC1/PCINT9)
- new net ADC2: U2.PC2(ADC2/PCINT10)
- new net ADC3: U2.PC3(ADC3/PCINT11)
- new net CH1: C9.2, J9.1, U3.CH1+
- new net CH2: C10.2, J9.2, U3.CH2+
- new net CH3: C11.2, J9.3, U3.CH3+
- new net CH4: C12.2, J9.4, U3.CH4+
- new net CH5: C14.2, J9.5, U4.CH1+
- new net CH6: C15.2, J9.6, U4.CH2+
- new net CH7: C16.2, J9.7, U4.CH3+
- new net CH8: C17.2, J9.8, U4.CH4+
- new net CTS: J4.5
- new net GPIO0: R2.2, U2.PD2(INT0/PCINT18)
- new net GPIO1: U2.PD3(PCINT19/OC2B/INT1)
- new net GPIO2: U2.PD4(PCINT20/XCK/T0)
- new net GPIO3: U2.PD5(PCINT21/OC0B/T1)
- new net GPIO4: U2.PD6(PCINT22/OC0A/AIN0)
- new net GPIO5: U2.PD7(PCINT23/AIN1)
- new net GPIO6: U2.PB0(PCINT0/CLKO/ICP1)
- new net GPIO7: U2.PB1(PCINT1/OC1A)
- new net MISO: J12.MISO, U2.PB4(PCINT4/MISO)
- new net MOSI: J12.MOSI, U2.PB3(PCINT3/OC2A/MOSI)
- new net N$3: D1.A, R2.1
- new net N$4: D2.A, R3.2
- new net N$5: C7.2, J4.1
- new net RST: C7.1, J12.RST, R1.1, SW1.B, U2.PC6(!RESET!/PCINT14)
- new net RX: J3.1, J4.3, U2.PD0(RXD/PCINT16)
- new net SCK: J12.SCK, U2.PB5(SCK/PCINT5)
- new net SS: U2.PB2(PCINT2/!SS!/OC1B)
- new net TX: J3.2, J4.2, U2.PD1(TXD/PCINT17)
- new net VCC: C1.2, J1.1, J1.2, J5.1, J5.2, U1.VIN
- new net XTAL1: C5.1, U2.PB6(PCINT6/XTAL1/TOSC1), Y1.B
- new net XTAL2: C6.1, U2.PB7(PCINT7/XTAL2/TOSC2), Y1.A
- net 5V: now also C13.2, C2.2, C3.2, C4.2, C8.2, J12.VCC, J4.4, R1.2, R3.1, R4.2, R5.2, TP1.P$1, U1.5V, U2.AVCC, U2.VCC, U3.VDD, U4.ADR1, U4.VDD; no longer C1.2, J6.1, J6.2, R2.2, R3.2, U1.VDD
- net GND: now also C10.1, C11.1, C12.1, C13.1, C14.1, C15.1, C16.1, C17.1, C2.1, C3.1, C4.1, C5.2, C6.2, C8.1, C9.1, D1.C, D2.C, J12.GND, J2.1, J4.6, J6.1, J6.2, SW1.A, U1.GND, U2.GND, U3.ADR0, U3.ADR1, U3.CH1-, U3.CH2-, U3.CH3-, U3.CH4-, U3.VSS, U4.ADR0, U4.CH1-, U4.CH2-, U4.CH3-, U4.CH4-, U4.VSS; no longer J5.1, J5.2, U1.ADR0, U1.ADR1, U1.VSS
- net SCL: now also J10.1, R5.1, U2.PC5(ADC5/SCL/PCINT13), U3.SCL, U4.SCL; no longer J4.1, R3.1, U1.SCL
- net SDA: now also J10.2, R4.1, U2.PC4(ADC4/SDA/PCINT12), U3.SDA, U4.SDA; no longer J4.2, R2.1, U1.SDA
