File: mippe_base_328_v2/mippe_base_v2.brd (EAGLE design)
At the start: 27 x 31.5 mm, 22 parts, among them J9 BURNIN, SW1 BTN-PTS810, U1 ATMEGA328P-AUR, Y1 16MHz

Commit message: update burnin drill size
Parts:
- turned D1 to 270 degrees
- turned D2 to 270 degrees
