File: mippe_mod/mippe_mod.sch (EAGLE design)
At the start: 21 parts, among them J1 VCC, J12 BURNIN, J3 UART, J4 FTDI, SW1 BTN-PTS810, U1 LM340MPX-5.0230, U2 ATMEGA328P-AUR, Y1 16MHz

Commit message: finish module and diff module
Parts:
- added J5: VCC, scono:CONN_02
- added J6: GND, scono:CONN_02
- added TP1: TEST_POINTTHRU, scono:TEST_POINTTHRU
- J2: value (none) -> GND
- R1: value (none) -> 10k
- R2, R3: value 330R -> 500R
Connections:
- net 5V: now also TP1.P$1; no longer U2.AREF
- net GND: now also J6.1, J6.2
- net VCC: now also J5.1, J5.2
Other:
- moved on the sheet: J3
Changed lines of the file:
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@@
 <part name="U1" library="scono" library_urn="urn:adsk.eagle:library:14850048" deviceset="LM340MPX-5.0" device="230" package3d_urn="urn:adsk.eagle:package:14850800/1"/>
 <part name="J1" library="scono" library_urn="urn:adsk.eagle:library:14850048" deviceset="CONN_02" device="" package3d_urn="urn:adsk.eagle:package:38039/1" value="VCC"/>
-<part name="J2" library="scono" library_urn="urn:adsk.eagle:library:14850048" deviceset="CONN_02" device="" package3d_urn="urn:adsk.eagle:package:38039/1"/>
+<part name="J2" library="scono" library_urn="urn:adsk.eagle:library:14850048" deviceset="CONN_02" device="" package3d_urn="urn:adsk.eagle:package:38039/1" value="GND"/>
 <part name="J3" library="scono" library_urn="urn:adsk.eagle:library:14850048" deviceset="CONN_02" device="" package3d_urn="urn:adsk.eagle:package:38039/1" value="UART"/>
 <part name="SUPPLY1" library="scono" library_urn="urn:adsk.eagle:library:14850048" deviceset="VCC" device=""/>
@@
 <attribute name="SUBSYSTEM_NAME" value="mippe_module"/>
 </part>
-<part name="R1" library="scono" library_urn="urn:adsk.eagle:library:14850048" deviceset="R-US_" device="R0402" package3d_urn="urn:adsk.eagle:package:14850590/2"/>
-<part name="R2" library="scono" library_urn="urn:adsk.eagle:library:14850048" deviceset="R-US_" device="R0402" package3d_urn="urn:adsk.eagle:package:14850590/2" value="330R"/>
+<part name="R1" library="scono" library_urn="urn:adsk.eagle:library:14850048" deviceset="R-US_" device="R0402" package3d_urn="urn:adsk.eagle:package:14850590/2" value="10k"/>
+<part name="R2" library="scono" library_urn="urn:adsk.eagle:library:14850048" deviceset="R-US_" device="R0402" package3d_urn="urn:adsk.eagle:package:14850590/2" value="500R"/>
 <part name="D1" library="scono" library_urn="urn:adsk.eagle:library:14850048" deviceset="LED" device="0603" package3d_urn="urn:adsk.eagle:package:14850721/2"/>
 <part name="SUPPLY6" library="scono" deviceset="GND" device=""/>
@@
 <part name="SUPPLY11" library="scono" deviceset="GND" device=""/>
 <part name="J4" library="scono" deviceset="CONN_06" device="NO_SILK_FEMALE_PTH" value="FTDI"/>
-<part name="R3" library="scono" library_urn="urn:adsk.eagle:library:14850048" deviceset="R-US_" device="R0402" package3d_urn="urn:adsk.eagle:package:14850590/2" value="330R"/>
+<part name="R3" library="scono" library_urn="urn:adsk.eagle:library:14850048" deviceset="R-US_" device="R0402" package3d_urn="urn:adsk.eagle:package:14850590/2" value="500R"/>
 <part name="D2" library="scono" library_urn="urn:adsk.eagle:library:14850048" deviceset="LED" device="0603" package3d_urn="urn:adsk.eagle:package:14850721/2" value="RED"/>
 <part name="SUPPLY13" library="scono" deviceset="GND" device=""/>
@@
 <part name="U$3" library="scono" library_urn="urn:adsk.eagle:library:14850048" deviceset="5V" device=""/>
 <part name="U$4" library="scono" library_urn="urn:adsk.eagle:library:14850048" deviceset="5V" device=""/>
+<part name="J5" library="scono" library_urn="urn:adsk.eagle:library:14850048" deviceset="CONN_02" device="" package3d_urn="urn:adsk.eagle:package:38039/1" value="VCC"/>
+<part name="SUPPLY12" library="scono" library_urn="urn:adsk.eagle:library:14850048" deviceset="VCC" device=""/>
+<part name="J6" library="scono" library_urn="urn:adsk.eagle:library:14850048" deviceset="CONN_02" device="" package3d_urn="urn:adsk.eagle:package:38039/1" value="GND"/>
+<part name="SUPPLY16" library="scono" library_urn="urn:adsk.eagle:library:14850048" deviceset="GND" device=""/>
+<part name="TP1" library="scono" library_urn="urn:adsk.eagle:library:14850048" deviceset="TEST_POINT" device="THRU" package3d_urn="urn:adsk.eagle:package:14850798/1"/>
 </parts>
 <sheets>
@@
 <attribute name="NAME" x="231.14" y="149.352" size="1.778" layer="95" font="vector" rot="R180"/>
 </instance>
-<instance part="J3" gate="G$1" x="228.6" y="167.64" smashed="yes" rot="R180">
-<attribute name="VALUE" x="231.14" y="172.466" size="1.778" layer="96" font="vector" rot="R180"/>
-<attribute name="NAME" x="231.14" y="162.052" size="1.778" layer="95" font="vector" rot="R180"/>
+<instance part="J3" gate="G$1" x="177.8" y="167.64" smashed="yes" rot="R180">
+<attribute name="VALUE" x="180.34" y="172.466" size="1.778" layer="96" font="vector" rot="R180"/>
+<attribute name="NAME" x="180.34" y="162.052" size="1.778" layer="95" font="vector" rot="R180"/>
 </instance>
 <instance part="SUPPLY1" gate="G$1" x="190.5" y="165.1" smashed="yes" rot="R90">
@@
 <instance part="U$4" gate="G$1" x="33.02" y="86.36" smashed="yes">
 <attribute name="VALUE" x="31.75" y="90.17" size="1.778" layer="96"/>
+</instance>
+<instance part="J5" gate="G$1" x="200.66" y="154.94" smashed="yes" rot="R180">
+<attribute name="VALUE" x="203.2" y="159.766" size="1.778" layer="96" font="vector" rot="R180"/>
+<attribute name="NAME" x="203.2" y="149.352" size="1.778" layer="95" font="vector" rot="R180"/>
+</instance>
+<instance part="SUPPLY12" gate="G$1" x="190.5" y="152.4" smashed="yes" rot="R90">
+<attribute name="VALUE" x="187.706" y="152.4" size="1.778" layer="96" rot="R90" align="bottom-center"/>
+</instance>
+<instance part="J6" gate="G$1" x="228.6" y="167.64" smashed="yes" rot="R180">
+<attribute name="VALUE" x="231.14" y="172.466" size="1.778" layer="96" font="vector" rot="R180"/>
+<attribute name="NAME" x="231.14" y="162.052" size="1.778" layer="95" font="vector" rot="R180"/>
+</instance>
+<instance part="SUPPLY16" gate="GND" x="215.9" y="165.1" smashed="yes" rot="R270">
+<attribute name="VALUE" x="213.36" y="166.37" size="1.016" layer="96" rot="R270"/>
+</instance>
+<instance part="TP1" gate="G$1" x="60.96" y="167.64" smashed="yes" rot="R90">
+<attribute name="NAME" x="58.42" y="167.64" size="1.778" layer="95" rot="R90"/>
 </instance>
 </instances>
@@
 <pinref part="SUPPLY5" gate="GND" pin="GND"/>
 </segment>
+<segment>
+<pinref part="J6" gate="G$1" pin="1"/>
+<pinref part="J6" gate="G$1" pin="2"/>
+<wire x1="220.98" y1="167.64" x2="220.98" y2="165.1" width="0.1524" layer="91"/>
+<wire x1="220.98" y1="165.1" x2="218.44" y2="165.1" width="0.1524" layer="91"/>
+<junction x="220.98" y="165.1"/>
+<pinref part="SUPPLY16" gate="GND" pin="GND"/>
+</segment>
 </net>
 <net name="SCL" class="0">
@@
 <segment>
 <pinref part="J3" gate="G$1" pin="1"/>
-<wire x1="220.98" y1="167.64" x2="218.44" y2="167.64" width="0.1524" layer="91"/>
-<label x="218.44" y="167.64" size="1.778" layer="95" rot="R180"/>
+<wire x1="170.18" y1="167.64" x2="167.64" y2="167.64" width="0.1524" layer="91"/>
+<label x="167.64" y="167.64" size="1.778" layer="95" rot="R180"/>
 </segment>
 </net>
@@
 <segment>
 <pinref part="J3" gate="G$1" pin="2"/>
-<wire x1="220.98" y1="165.1" x2="218.44" y2="165.1" width="0.1524" layer="91"/>
-<label x="218.44" y="165.1" size="1.778" layer="95" rot="R180"/>
+<wire x1="170.18" y1="165.1" x2="167.64" y2="165.1" width="0.1524" layer="91"/>
+<label x="167.64" y="165.1" size="1.778" layer="95" rot="R180"/>
 </segment>
 </net>
@@
 <wire x1="134.62" y1="111.76" x2="134.62" y2="109.22" width="0.1524" layer="91"/>
 <junction x="134.62" y="111.76"/>
-<pinref part="U2" gate="G$1" pin="AREF"/>
-<wire x1="134.62" y1="109.22" x2="134.62" y2="106.68" width="0.1524" layer="91"/>
-<junction x="134.62" y="109.22"/>
 </segment>
 <segment>
@@
 <wire x1="60.96" y1="167.64" x2="60.96" y2="165.1" width="0.1524" layer="91"/>
 <junction x="60.96" y="167.64"/>
+<pinref part="TP1" gate="G$1" pin="P$1"/>
 </segment>
 <segment>
@@
 <junction x="25.4" y="167.64"/>
 </segment>
-</net>
+<segment>
+<pinref part="J5" gate="G$1" pin="2"/>
+<pinref part="J5" gate="G$1" pin="1"/>
+<wire x1="193.04" y1="152.4" x2="193.04" y2="154.94" width="0.1524" layer="91"/>
+<wire x1="193.04" y1="152.4" x2="190.5" y2="152.4" width="0.1524" layer="91"/>
+<junction x="193.04" y="152.4"/>
+<pinref part="SUPPLY12" gate="G$1" pin="VCC"/>
+</segment>
+</net>

Commit message: finish bom cpl for mippe mod and adc diff
Parts:
- C7: value 0.1uF -> 100nF
Changed lines of the file:
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@@
 <part name="U2" library="scono" deviceset="ATMEGA328P-AUR" device=""/>
 <part name="SUPPLY15" library="scono" deviceset="GND" device=""/>
-<part name="C7" library="scono" library_urn="urn:adsk.eagle:library:14850048" deviceset="CAP" device="0402-CAP" package3d_urn="urn:adsk.eagle:package:14850678/2" value="0.1uF"/>
+<part name="C7" library="scono" library_urn="urn:adsk.eagle:library:14850048" deviceset="CAP" device="0402-CAP" package3d_urn="urn:adsk.eagle:package:14850678/2" value="100nF"/>
 <part name="U$2" library="scono" library_urn="urn:adsk.eagle:library:14850048" deviceset="5V" device=""/>
 <part name="U$5" library="scono" library_urn="urn:adsk.eagle:library:14850048" deviceset="5V" device=""/>
