File: mippe_mod_test/mippe_mod_test.brd (EAGLE design)
At the start: 32.5 x 50 mm, 24 parts, among them J1 VCC, J12 BURNIN, J2 GND, J3 UART, J4 FTDI, J5 VCC, J6 GND, SW1 BTN-PTS810, U1 LM340MPX-5.0230, U2 ATMEGA328P-AUR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

Commit message: blaaahhhhh 328pb worked
Parts:
- added TP10, TP2, TP3, TP4, TP5, TP6, TP7, TP8, TP9: TEST_POINTTHRU, scono:TEST_POINT
Connections:
- net MISO: now also TP3.1
- net MOSI: now also TP4.1
- net N$3: now also TP8.1
- net RST: now also TP5.1
- net RX: now also TP7.1
- net SCK: now also TP2.1
- net TX: now also TP6.1
- net XTAL1: now also TP9.1
- net XTAL2: now also TP10.1
Routing:
- net TX: track 16.5 -> 50.9 mm, vias 2 -> 3
- net N$3: track 16.5 -> 47.7 mm, vias 0 -> 1
- net RST: track 26.2 -> 55.2 mm, vias 1 -> 3
- net RX: track 15.5 -> 37.8 mm, vias 2 -> 3
- net SCK: track 26.3 -> 46.1 mm
- net MISO: track 26.7 -> 39.8 mm
- net XTAL1: track 10.7 -> 21.9 mm, vias 0 -> 1
- net XTAL2: track 7.89 -> 17.1 mm, vias 0 -> 2
- net MOSI: track 24.8 -> 32.3 mm
Other:
- board text added: "DTR"
- board text added: "MISO"
- board text added: "MOSI"
- board text added: "RST"
- board text added: "RX"
- board text added: "SCK"
- board text added: "TX"
