File: board tester oled transimp/opd tester.sch (EAGLE design)
At the start: 18 parts, among them IC1 TL7660, J1 i2c, U1 MCP4725A0T-E/CH, U2 LMC6482AIM/NOPB

Commit message: more work
Parts:
- removed TP2: TEST_POINTTHRU, scono:TEST_POINTTHRU
- added R4, R5: 10k, scono:R-US_0603
Connections:
- net 5V: now also R4.2, R5.1
- net OUTSIG: no longer TP2.P$1
- net SCL: now also R4.1
- net SDA: now also R5.2
Changed lines of the file:
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@@
 <part name="J3" library="scono" library_urn="urn:adsk.eagle:library:14850048" deviceset="CONN_02" device="" package3d_urn="urn:adsk.eagle:package:38039/1"/>
 <part name="TP1" library="scono" library_urn="urn:adsk.eagle:library:14850048" deviceset="TEST_POINT" device="THRU" package3d_urn="urn:adsk.eagle:package:14850798/1"/>
-<part name="TP2" library="scono" library_urn="urn:adsk.eagle:library:14850048" deviceset="TEST_POINT" device="THRU" package3d_urn="urn:adsk.eagle:package:14850798/1"/>
 <part name="TP3" library="scono" library_urn="urn:adsk.eagle:library:14850048" deviceset="TEST_POINT" device="THRU" package3d_urn="urn:adsk.eagle:package:14850798/1"/>
 <part name="TP4" library="scono" library_urn="urn:adsk.eagle:library:14850048" deviceset="TEST_POINT" device="THRU" package3d_urn="urn:adsk.eagle:package:14850798/1"/>
 <part name="TP5" library="scono" library_urn="urn:adsk.eagle:library:14850048" deviceset="TEST_POINT" device="THRU" package3d_urn="urn:adsk.eagle:package:14850798/1"/>
 <part name="U$5" library="scono" library_urn="urn:adsk.eagle:library:14850048" deviceset="5V" device=""/>
+<part name="R4" library="scono" library_urn="urn:adsk.eagle:library:14850048" deviceset="R-US_" device="0603" package3d_urn="urn:adsk.eagle:package:14850803/1" value="10k"/>
+<part name="R5" library="scono" library_urn="urn:adsk.eagle:library:14850048" deviceset="R-US_" device="0603" package3d_urn="urn:adsk.eagle:package:14850803/1" value="10k"/>
+<part name="U$6" library="scono" library_urn="urn:adsk.eagle:library:14850048" deviceset="5V" device=""/>
+<part name="U$7" library="scono" library_urn="urn:adsk.eagle:library:14850048" deviceset="5V" device=""/>
 </parts>
 <sheets>
@@
 <attribute name="NAME" x="86.36" y="83.82" size="1.778" layer="95" rot="R270"/>
 </instance>
-<instance part="TP2" gate="G$1" x="200.66" y="114.3" smashed="yes" rot="R90">
-<attribute name="NAME" x="198.12" y="114.3" size="1.778" layer="95" rot="R90"/>
-</instance>
 <instance part="TP3" gate="G$1" x="215.9" y="111.76" smashed="yes" rot="R270">
 <attribute name="NAME" x="218.44" y="111.76" size="1.778" layer="95" rot="R270"/>
@@
 <instance part="U$5" gate="G$1" x="83.82" y="160.02" smashed="yes">
 <attribute name="VALUE" x="82.55" y="163.83" size="1.778" layer="96"/>
+</instance>
+<instance part="R4" gate="G$1" x="27.94" y="149.86" smashed="yes" rot="R90">
+<attribute name="NAME" x="26.67" y="144.78" size="1.016" layer="95" rot="R90"/>
+<attribute name="VALUE" x="29.21" y="144.78" size="1.016" layer="96" rot="R90" align="top-left"/>
+</instance>
+<instance part="R5" gate="G$1" x="33.02" y="139.7" smashed="yes" rot="R90">
+<attribute name="NAME" x="31.75" y="134.62" size="1.016" layer="95" rot="R90"/>
+<attribute name="VALUE" x="34.29" y="134.62" size="1.016" layer="96" rot="R90" align="top-left"/>
+</instance>
+<instance part="U$6" gate="G$1" x="27.94" y="152.4" smashed="yes">
+<attribute name="VALUE" x="26.67" y="156.21" size="1.778" layer="96"/>
+</instance>
+<instance part="U$7" gate="G$1" x="33.02" y="134.62" smashed="yes" rot="R180">
+<attribute name="VALUE" x="34.29" y="130.81" size="1.778" layer="96" rot="R180"/>
 </instance>
 </instances>
@@
 <pinref part="J1" gate="G$1" pin="2"/>
 <pinref part="U1" gate="G$1" pin="SCL"/>
-<wire x1="25.4" y1="144.78" x2="48.26" y2="144.78" width="0.1524" layer="91"/>
+<wire x1="25.4" y1="144.78" x2="27.94" y2="144.78" width="0.1524" layer="91"/>
 <label x="35.56" y="144.78" size="1.778" layer="95"/>
+<pinref part="R4" gate="G$1" pin="1"/>
+<wire x1="27.94" y1="144.78" x2="48.26" y2="144.78" width="0.1524" layer="91"/>
+<junction x="27.94" y="144.78"/>
 </segment>
 </net>
@@
 <pinref part="J1" gate="G$1" pin="1"/>
 <pinref part="U1" gate="G$1" pin="SDA"/>
-<wire x1="25.4" y1="142.24" x2="48.26" y2="142.24" width="0.1524" layer="91"/>
+<wire x1="25.4" y1="142.24" x2="33.02" y2="142.24" width="0.1524" layer="91"/>
+<wire x1="33.02" y1="142.24" x2="48.26" y2="142.24" width="0.1524" layer="91"/>
 <wire x1="48.26" y1="142.24" x2="48.26" y2="139.7" width="0.1524" layer="91"/>
 <label x="35.56" y="139.7" size="1.778" layer="95"/>
+<pinref part="R5" gate="G$1" pin="2"/>
+<junction x="33.02" y="142.24"/>
 </segment>
 </net>
@@
 <pinref part="U1" gate="G$1" pin="VDD"/>
 <wire x1="83.82" y1="160.02" x2="83.82" y2="154.94" width="0.1524" layer="91"/>
+</segment>
+<segment>
+<pinref part="R4" gate="G$1" pin="2"/>
+<pinref part="U$6" gate="G$1" pin="5V"/>
+</segment>
+<segment>
+<pinref part="R5" gate="G$1" pin="1"/>
+<pinref part="U$7" gate="G$1" pin="5V"/>
 </segment>
 </net>
@@
 <junction x="200.66" y="101.6"/>
 <label x="210.82" y="101.6" size="1.778" layer="95"/>
-<pinref part="TP2" gate="G$1" pin="P$1"/>
-</segment>
-<segment>
+</segment>
+<segment>

Commit message: add cap for stabalization
Parts:
- added C4: 0.1uF, scono:CAP0603-CAP
Connections:
- net N$3: now also C4.1
- net N$4: now also C4.2
Changed lines of the file:
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@@
 <part name="U$6" library="scono" library_urn="urn:adsk.eagle:library:14850048" deviceset="5V" device=""/>
 <part name="U$7" library="scono" library_urn="urn:adsk.eagle:library:14850048" deviceset="5V" device=""/>
+<part name="C4" library="scono" library_urn="urn:adsk.eagle:library:14850048" deviceset="CAP" device="0603-CAP" package3d_urn="urn:adsk.eagle:package:14850677/1" value="0.1uF"/>
 </parts>
 <sheets>
@@
 <attribute name="VALUE" x="34.29" y="130.81" size="1.778" layer="96" rot="R180"/>
 </instance>
+<instance part="C4" gate="G$1" x="104.14" y="119.38" smashed="yes" rot="R90">
+<attribute name="NAME" x="102.616" y="118.11" size="1.016" layer="95" rot="R90"/>
+<attribute name="VALUE" x="106.68" y="118.11" size="1.016" layer="96" rot="R90"/>
+</instance>
 </instances>
 <busses>
@@
 <pinref part="TP5" gate="G$1" pin="P$1"/>
 <junction x="116.84" y="114.3"/>
+<pinref part="C4" gate="G$1" pin="1"/>
+<wire x1="104.14" y1="116.84" x2="104.14" y2="114.3" width="0.1524" layer="91"/>
+<wire x1="104.14" y1="114.3" x2="109.22" y2="114.3" width="0.1524" layer="91"/>
 </segment>
 </net>
@@
 <pinref part="R2" gate="G$1" pin="2"/>
 <pinref part="TP4" gate="G$1" pin="P$1"/>
-</segment>
-</net>
+<pinref part="C4" gate="G$1" pin="2"/>
+<wire x1="104.14" y1="121.92" x2="109.22" y2="121.92" width="0.1524" layer="91"/>
+<junction x="109.22" y="121.92"/>
+</segment>
+</net>
