File: pas_pot_diff/pas_pot_diff.brd (EAGLE design)
At the start: 32.5 x 50 mm, 37 parts, among them J1 VCC, J10 I2C, J12 BURNIN, J2 GND, J3 UART, J4 FTDI, J5 VCC, J6 GND, SW1 BTN-PTS810, U1 LM340MPX-5.0230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

Commit message: update burnin drill size
Routing:
- net GND: track 74.8 -> 73.5 mm
Changed lines of the file:
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@@
 <attribute name="PIE-INT-REF-NUM" value="CAPACITOR-GENERIC" x="11.75" y="42.25" size="1.778" layer="27" rot="R180" display="off"/>
 </element>
-<element name="U4" library="scono" library_urn="urn:adsk.eagle:library:14850048" package="RU_24" value="AD8403ARUZ100" x="22.75" y="37" smashed="yes" rot="R180">
+<element name="U4" library="scono" library_urn="urn:adsk.eagle:library:14850048" package="RU_24" package3d_urn="urn:adsk.eagle:package:17602555/1" value="AD8403ARUZ100" x="22.75" y="37" smashed="yes" rot="R180">
 <attribute name="BUILT_BY" value="EMA_UL_Team" x="22.75" y="37" size="1.778" layer="27" rot="R180" display="off"/>
 <attribute name="MANUFACTURER_PART_NUMBER" value="AD8403ARUZ100" x="22.75" y="37" size="1.778" layer="27" rot="R180" display="off"/>
@@
 <contactref element="U4" pad="21"/>
 <contactref element="C13" pad="1"/>
-<wire x1="20.725" y1="39.275" x2="21.25" y2="38.75" width="0.1" layer="1"/>
-<wire x1="21.25" y1="38.75" x2="21.25" y2="38.25" width="0.1" layer="1"/>
 <wire x1="21.25" y1="38.25" x2="20.975" y2="37.975" width="0.1" layer="1"/>
 <wire x1="20.975" y1="37.975" x2="19.9306" y2="37.975" width="0.1" layer="1"/>

Commit message: finish transimp module
Other:
- board text added: "Passive Potentiometric Sensor Module"
Changed lines of the file:
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@@
 <text x="12.5" y="44" size="0.7" layer="21" rot="SR180">Ch4</text>
 <text x="16.25" y="49.25" size="1" layer="21" font="vector" rot="SR180" align="bottom-center">Plug other side to GND</text>
+<text x="10" y="46" size="1" layer="21" rot="SR180">Passive
+Potentiometric
+Sensor
+Module</text>
 </plain>
 <attributes>
@@
 </drawing>
 <compatibility>
+<note version="6.3" minversion="6.2.2" severity="warning">
+Since Version 6.2.2 text objects can contain more than one line,
+which will not be processed correctly with this version.
+</note>
 <note version="8.2" severity="warning">
 Since Version 8.2, EAGLE supports online libraries. The ids
