File: transimp/transimp.brd (EAGLE design)
At the start: 32.5 x 50 mm, 33 parts, among them J1 VCC, J12 BURNIN, J2 GND, J3 UART, J4 FTDI, J5 VCC, J6 GND, SW1 BTN-PTS810, U1 LM340MPX-5.0230, U2 ATMEGA328P-AUR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

Commit message: finish transimp module
Parts:
- removed TP10, TP3, TP4, TP5, TP6, TP7, TP8, TP9: TEST_POINTTHRU, scono:TEST_POINT
- added C10, C11, C12, C13: 0.1uF, scono:0402-CAP
- added C8, C9: 10uF, scono:CAP_3MM
- added IC1: TL7660, scono:8SOICW
- added J7: i2c, scono:1X02
- added J8: (no value), scono:1X04
- added R10, R11, R4, R5, R6, R9: 100k, scono:R0402
- added R7, R8: 10k, scono:R0402
- added U3, U5: MCP4725A0T-E/CH, scono:SOT95P270X145-6N
- added U4, U6: LMC6482AIM/NOPB, scono:M08A
- moved TP2 22.9 mm to (30.2, 28.2)
Connections:
- removed net ADC1: U2.24
- removed net ADC2: U2.25
- new net -5V: C9.NEG, IC1.5, TP2.1, U4.4, U6.4
- new net ANODE1: C11.1, J8.1, R4.1, U4.2
- new net ANODE2: C13.1, J8.3, R9.1, U6.2
- new net CATHODE1: J8.2, U3.1
- new net CATHODE2: J8.4, U5.1
- new net N$4: C8.POS, IC1.2
- new net N$5: C8.NEG, IC1.4
- new net N$6: C13.2, R10.2, R9.2, U6.1
- new net N$7: C11.2, R4.2, R5.2, U4.1
- new net N$8: R5.1, R6.1, U4.6
- new net N$9: R10.1, R11.1, U6.6
- new net OUTSIG$1: C10.2, R6.2, U2.24, U4.7
- new net OUTSIG$2: C12.2, R11.2, U2.25, U6.7
- net 5V: now also IC1.8, R7.2, R8.1, U3.3, U4.8, U5.3, U5.6, U6.8
- net GND: now also C10.1, C12.1, C9.POS, IC1.3, U3.2, U3.6, U4.3, U4.5, U5.2, U6.3, U6.5
- net MISO: no longer TP3.1
- net MOSI: no longer TP4.1
- net N$3: no longer TP8.1
- net RST: no longer TP5.1
- net RX: no longer TP7.1
- net SCK: no longer TP2.1
- net SCL: now also J7.2, R7.1, U3.5, U5.5
- net SDA: now also J7.1, R8.2, U3.4, U5.4
- net TX: no longer TP6.1
- net XTAL1: no longer TP9.1
- net XTAL2: no longer TP10.1
Routing:
- net SCL: track 0.00 -> 42.4 mm, vias 0 -> 5
- net SDA: track 0.00 -> 41.8 mm, vias 0 -> 5
- net OUTSIG$2: track 0.00 -> 35.1 mm, vias 0 -> 4
- net TX: track 50.9 -> 16.5 mm, vias 3 -> 2
- net -5V: track 0.00 -> 33.5 mm, vias 0 -> 1
- net N$3: track 47.7 -> 16.5 mm, vias 1 -> 0
- net RST: track 55.2 -> 26.2 mm, vias 3 -> 1
- net OUTSIG$1: track 0.00 -> 28.8 mm, vias 0 -> 2
- net CATHODE1: track 0.00 -> 23.6 mm, vias 0 -> 2
- net RX: track 37.8 -> 15.5 mm, vias 3 -> 2
- net CATHODE2: track 0.00 -> 20.2 mm, vias 0 -> 2
- net SCK: track 46.1 -> 26.3 mm
- net N$6: track 0.00 -> 17.2 mm, vias 0 -> 2
- net N$7: track 0.00 -> 17.2 mm, vias 0 -> 2
- net ANODE1: track 0.00 -> 14.2 mm, vias 0 -> 1
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Other:
- board text added: "PD1"
- board text added: "PD2"
- board text added: "Transimp Amplifier Module"
- board text removed: "DTR"
- board text removed: "MISO"
- board text removed: "MOSI"
- board text removed: "RST"
- board text removed: "RX"
- board text removed: "SCK"
- board text removed: "TX"
