File: transimp/transimp.sch (EAGLE design)
At the start: 33 parts, among them J1 VCC, J12 BURNIN, J2 GND, J3 UART, J4 FTDI, J5 VCC, J6 GND, SW1 BTN-PTS810, U1 LM340MPX-5.0230, U2 ATMEGA328P-AUR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

Commit message: finish transimp module
Parts:
- removed TP10, TP3, TP4, TP5, TP6, TP7, TP8, TP9: TEST_POINTTHRU, scono:TEST_POINTTHRU
- added C10, C11, C12, C13: 0.1uF, scono:CAP0402-CAP
- added C8, C9: 10uF, scono:CAP_ELEC_3MM_SMD
- added IC1: TL7660, scono:TL7660
- added J7: i2c, scono:CONN_02
- added J8: (no value), scono:CONN_04
- added R10, R11, R4, R5, R6, R9: 100k, scono:R-US_R0402
- added R7, R8: 10k, scono:R-US_R0402
- added U3, U5: MCP4725A0T-E/CH, scono:MCP4725A0T-E/CH
- added U4, U6: LMC6482AIM/NOPB, scono:LMC6482AIM/NOPB
Connections:
- removed net ADC1: U2.PC1(ADC1/PCINT9)
- removed net ADC2: U2.PC2(ADC2/PCINT10)
- new net -5V: C9.NEG, IC1.VOUT, TP2.P$1, U4.VCC-, U6.VCC-
- new net ANODE1: C11.1, J8.1, R4.1, U4.INPUT1-
- new net ANODE2: C13.1, J8.3, R9.1, U6.INPUT1-
- new net CATHODE1: J8.2, U3.VOUT
- new net CATHODE2: J8.4, U5.VOUT
- new net N$4: C8.POS, IC1.CAP+
- new net N$5: C8.NEG, IC1.CAP-
- new net N$6: C13.2, R10.2, R9.2, U6.OUT1
- new net N$7: C11.2, R4.2, R5.2, U4.OUT1
- new net N$8: R5.1, R6.1, U4.INPUT2-
- new net N$9: R10.1, R11.1, U6.INPUT2-
- new net OUTSIG$1: C10.2, R6.2, U2.PC1(ADC1/PCINT9), U4.OUT2
- new net OUTSIG$2: C12.2, R11.2, U2.PC2(ADC2/PCINT10), U6.OUT2
- net 5V: now also IC1.VCC, R7.2, R8.1, U3.VDD, U4.VCC+, U5.A0, U5.VDD, U6.VCC+
- net GND: now also C10.1, C12.1, C9.POS, IC1.GND, U3.A0, U3.VSS, U4.INPUT1+, U4.INPUT2+, U5.VSS, U6.INPUT1+, U6.INPUT2+
- net MISO: no longer TP3.P$1
- net MOSI: no longer TP4.P$1
- net N$3: no longer TP8.P$1
- net RST: no longer TP5.P$1
- net RX: no longer TP7.P$1
- net SCK: no longer TP2.P$1
- net SCL: now also J7.2, R7.1, U3.SCL, U5.SCL
- net SDA: now also J7.1, R8.2, U3.SDA, U5.SDA
- net TX: no longer TP6.P$1
- net XTAL1: no longer TP9.P$1
- net XTAL2: no longer TP10.P$1
