File: mippe_mobo_v2/mippe_mobo.brd (EAGLE design)
At the start: 120 x 120 mm, 29 parts, among them J3 FFC-32, J4 PJ-102AH, U1 CD4052BPWR, U2 MIPPE, U3 LM340MPX-5.0230

Commit message: place final order for mobo
Connections:
- net GND: now also J4.2; no longer J4.1
- net VCC: now also J4.1; no longer J4.2
Routing:
- net GND: track 323.4 -> 316.6 mm
- net VCC: track 279.9 -> 276.4 mm
Changed lines of the file:
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@@
 <wire x1="50" y1="64.75" x2="50" y2="78.5" width="1.25" layer="1"/>
 <via x="50" y="78.5" extent="1-16" drill="1.25" diameter="1"/>
-<contactref element="J4" pad="2"/>
 <contactref element="C8" pad="POS"/>
-<contactref element="TP4" pad="1"/>
-<wire x1="60" y1="114.75" x2="57.75" y2="117" width="0.5" layer="1"/>
-<wire x1="57.75" y1="117" x2="50.25" y2="117" width="0.5" layer="1"/>
-<wire x1="60" y1="114.75" x2="63.5" y2="111.25" width="1" layer="1"/>
-<wire x1="63.5" y1="106.35" x2="61.9" y2="104.75" width="1" layer="1"/>
-<wire x1="63.5" y1="111.25" x2="63.5" y2="106.35" width="1" layer="1"/>
 <wire x1="50" y1="78.5" x2="50" y2="92.5" width="1.25" layer="16"/>
 <wire x1="50" y1="92.5" x2="45.25" y2="97.25" width="1.25" layer="16"/>
@@
 <wire x1="45.25" y1="97.25" x2="45.25" y2="105.5" width="1.25" layer="1"/>
 <wire x1="45.25" y1="105.5" x2="45.25" y2="114.25" width="1.25" layer="1"/>
-<wire x1="48" y1="117" x2="50.25" y2="117" width="1.25" layer="1"/>
-<wire x1="45.25" y1="114.25" x2="48" y2="117" width="1.25" layer="1"/>
+<wire x1="48" y1="117" x2="45.25" y2="114.25" width="1.25" layer="1"/>
 <contactref element="U3" pad="1"/>
 <wire x1="48.925" y1="107.55" x2="47.3" y2="107.55" width="0.5" layer="1"/>
 <wire x1="47.3" y1="107.55" x2="45.25" y2="105.5" width="0.5" layer="1"/>
+<contactref element="J4" pad="1"/>
+<contactref element="TP4" pad="1"/>
+<wire x1="60" y1="108.75" x2="58.25" y2="110.5" width="1.25" layer="1"/>
+<wire x1="54" y1="117" x2="50.25" y2="117" width="1.25" layer="1"/>
+<wire x1="58.25" y1="110.5" x2="58.25" y2="112.75" width="1.25" layer="1"/>
+<wire x1="58.25" y1="112.75" x2="54" y2="117" width="1.25" layer="1"/>
+<wire x1="50.25" y1="117" x2="48" y2="117" width="1.25" layer="1"/>
+<wire x1="60" y1="108.75" x2="61.9" y2="106.85" width="1.25" layer="1"/>
+<wire x1="61.9" y1="106.85" x2="61.9" y2="104.75" width="1.25" layer="1"/>
 </signal>
 <signal name="GND">
@@
 <contactref element="B1" pad="GND@3"/>
 <via x="60.35" y="100.5" extent="1-16" drill="0.2"/>
-<contactref element="J4" pad="1"/>
-<contactref element="J4" pad="3"/>
-<wire x1="55.3" y1="111.75" x2="56" y2="111.75" width="1" layer="16"/>
-<wire x1="56" y1="111.75" x2="57" y2="111.75" width="1" layer="16"/>
-<wire x1="57" y1="111.75" x2="60" y2="108.75" width="1" layer="16"/>
 <contactref element="J6" pad="1"/>
 <contactref element="J6" pad="2"/>
@@
 <contactref element="U2" pad="GND@1"/>
 <wire x1="73.07" y1="114.215" x2="73.07" y2="116.755" width="1" layer="16"/>
-<wire x1="50.25" y1="113.75" x2="52.25" y2="111.75" width="1" layer="16"/>
-<wire x1="52.25" y1="111.75" x2="56" y2="111.75" width="1" layer="16"/>
-<wire x1="60" y1="108.75" x2="58.1" y2="106.85" width="1" layer="1"/>
-<wire x1="58.1" y1="106.85" x2="58.1" y2="104.75" width="1" layer="1"/>
 <wire x1="46" y1="70.54" x2="46" y2="83" width="1.25" layer="16"/>
 <wire x1="42.5" y1="86.5" x2="42.5" y2="107.25" width="1.25" layer="16"/>
@@
 <wire x1="55.075" y1="105.25" x2="55.575" y2="104.75" width="0.5" layer="1"/>
 <wire x1="55.575" y1="104.75" x2="58.1" y2="104.75" width="0.5" layer="1"/>
-<wire x1="60" y1="108.75" x2="65.465" y2="114.215" width="1.25" layer="16"/>
-<wire x1="65.465" y1="114.215" x2="73.07" y2="114.215" width="1.25" layer="16"/>
+<contactref element="J4" pad="2"/>
+<contactref element="J4" pad="3"/>
+<wire x1="60.535" y1="114.215" x2="60" y2="114.75" width="1.25" layer="16"/>
+<wire x1="73.07" y1="114.215" x2="60.535" y2="114.215" width="1.25" layer="16"/>
+<wire x1="60" y1="114.75" x2="57" y2="111.75" width="1.25" layer="16"/>
+<wire x1="57" y1="111.75" x2="55.3" y2="111.75" width="1.25" layer="16"/>
+<wire x1="55.075" y1="105.25" x2="55.075" y2="111.525" width="1.25" layer="1"/>
+<wire x1="55.075" y1="111.525" x2="55.3" y2="111.75" width="1.25" layer="1"/>
 </signal>
 <signal name="TX1">
@@
 <contactref element="U3" pad="3"/>
 <contactref element="C2" pad="2"/>
-<contactref element="C2" pad="2"/>
-</signal>
+</signal>
