File: mippe_mobo_v2/mippe_mobo.sch (EAGLE design)
At the start: 53 parts, among them J3 FFC-32, J4 PJ-102AH, J5 BURNIN, SW1 BTN-PTS810, U1 CD4052BPWR, U3 ATMEGA32U4-XUMU, X1 USB-B1HSB6, Y1 16MHz

Commit message: finalize mobo
Parts:
- removed C10, C9: 18pF, scono:CAP0402-CAP
- removed C3, C4: 0.1uF, scono:CAP0402-CAP
- removed C5, C6, C7: 1uF, scono:CAP0402-CAP
- removed D1, D2, D3: (no value), scono:LED0603
- removed F1: 500mA, scono:0ZCJ0050FF2G1206
- removed J5: BURNIN, scono:BURNIN
- removed L2: (no value), scono:IND
- removed R10, R9: 10k, scono:R-US_R0402
- removed R11, R12, R15: 330R, scono:R-US_R0402
- removed R7, R8: 22R, scono:R-US_R0402
- removed SW1: BTN-PTS810, scono:BTN-PTS810
- removed TP5: TEST_POINTTHRU, scono:TEST_POINTTHRU
- removed X1: USB-B1HSB6, scono:USB-B1HSB6
- removed Y1: 16MHz, scono:CRYSTAL_SMOL
- removed Z1, Z2: CG0603MLC-05E, scono:VARISTOR
- added U2: MIPPE, scono:MIPPE
- C2: device scono:CAP0402-CAP -> scono:CAP0603-CAP
- U3: value ATMEGA32U4-XUMU -> LM340MPX-5.0230; device scono:ATMEGA32U4-XUMU -> scono:LM340MPX-5.0230
Connections:
- removed net AGND: C3.1, L2.P$2, U3.GND3
- removed net AREF: C3.2, U3.AREF
- removed net D_N: R7.1, X1.D-, Z2.1
- removed net D_P: R8.1, X1.D+, Z1.1
- removed net HWB: R9.1, U3.(#HWB)PE2
- removed net MISO: J5.MISO, U3.(PD0/MISO/PCINT3)PB3
- removed net MOSI: J5.MOSI, U3.(PDI/MOSI/PCINT2)PB2
- removed net N$33: D2.C, R11.2
- removed net N$34: D3.C, R12.2
- removed net N$35: D1.C, R15.2
- removed net RD_N: R7.2, U3.D-
- removed net RD_P: R8.2, U3.D+
- removed net RESET: J5.RST, R10.1, SW1.B, U3.RESET
- removed net RXLED: R12.1, U3.(SS/PCINT0)PB0
- removed net SCK: J5.SCK, U3.(SCLK/PCINT1)PB1
- removed net TXLED: R11.1, U3.(XCK1/#CTS)PD5
- removed net UCAP: C7.2, U3.UCAP
- removed net XTAL1: C9.2, U3.XTAL1, Y1.A
- removed net XTAL2: C10.2, U3.XTAL2, Y1.B
- removed net XUSB: F1.1, X1.VCC
- net 5V: now also U3.5V; no longer C4.2, C5.2, C6.2, D1.A, D2.A, D3.A, F1.2, J5.VCC, R10.2, TP5.P$1, U3.AVCC, U3.AVCC1, U3.UVCC, U3.VBUS, U3.VCC, U3.VCC1
- net A: now also U2.GPIO5; no longer U3.(OC0B/SCL/INT0)PD0
- net B: now also U2.GPIO4; no longer U3.(SDA/INT1)PD1
- net GND: now also U2.GND; no longer C10.1, C4.1, C5.1, C6.1, C7.1, C9.1, J5.GND, L2.P$1, R15.1, R9.2, SW1.A, U3.GND1, U3.GND2, U3.PAD, U3.UGND, X1.GND, Z1.2, Z2.2
- net RX: now also U2.RX; no longer U3.(RXD1/AIN1/INT2)PD2
- net TX: now also U2.TX; no longer U3.(TXD1/INT3)PD3
- net VCC: now also U3.VIN

Commit message: place final order for mobo
Connections:
- net GND: now also J4.2; no longer J4.1
- net VCC: now also J4.1; no longer J4.2
Other:
- moved on the sheet: TP4
Changed lines of the file:
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@@
 <part name="L1" library="scono" library_urn="urn:adsk.eagle:library:14850048" deviceset="UCB_CAL" device="500MIL" value="UCB_CAL500MIL"/>
 <part name="J4" library="scono" library_urn="urn:adsk.eagle:library:14850048" deviceset="PJ-102AH" device=""/>
-<part name="SUPPLY7" library="scono" library_urn="urn:adsk.eagle:library:14850048" deviceset="GND" device=""/>
-<part name="SUPPLY8" library="scono" library_urn="urn:adsk.eagle:library:14850048" deviceset="VCC" device=""/>
 <part name="J6" library="scono" library_urn="urn:adsk.eagle:library:14850048" deviceset="CONN_04" device="" package3d_urn="urn:adsk.eagle:package:38085/1"/>
 <part name="SUPPLY9" library="scono" library_urn="urn:adsk.eagle:library:14850048" deviceset="GND" device=""/>
@@
 <part name="C2" library="scono" library_urn="urn:adsk.eagle:library:14850048" deviceset="CAP" device="0603-CAP" package3d_urn="urn:adsk.eagle:package:14850677/1" value="0.1uF"/>
 <part name="SUPPLY17" library="scono" library_urn="urn:adsk.eagle:library:14850048" deviceset="GND" device=""/>
+<part name="SUPPLY7" library="scono" library_urn="urn:adsk.eagle:library:14850048" deviceset="VCC" device=""/>
+<part name="SUPPLY8" library="scono" library_urn="urn:adsk.eagle:library:14850048" deviceset="GND" device=""/>
 </parts>
 <sheets>
@@
 <attribute name="VALUE" x="99.05045" y="160.01363125" size="1.78023125" layer="96"/>
 </instance>
-<instance part="SUPPLY7" gate="GND" x="127" y="167.64" smashed="yes" rot="R90"/>
-<instance part="SUPPLY8" gate="G$1" x="124.46" y="162.56" smashed="yes" rot="R270">
-<attribute name="VALUE" x="127.254" y="162.56" size="1.778" layer="96" rot="R270" align="bottom-center"/>
-</instance>
 <instance part="C8" gate="G$1" x="139.7" y="165.1" smashed="yes">
 <attribute name="NAME" x="140.716" y="165.735" size="1.778" layer="95"/>
@@
 <attribute name="NAME" x="48.26" y="50.8" size="1.778" layer="95" rot="R180"/>
 </instance>
-<instance part="TP4" gate="G$1" x="121.92" y="162.56" smashed="yes" rot="R270">
-<attribute name="NAME" x="124.46" y="162.56" size="1.778" layer="95" rot="R270"/>
+<instance part="TP4" gate="G$1" x="119.38" y="167.64" smashed="yes" rot="R90">
+<attribute name="NAME" x="116.84" y="167.64" size="1.778" layer="95" rot="R90"/>
 </instance>
 <instance part="R13" gate="G$1" x="177.8" y="53.34" smashed="yes" rot="R270">
@@
 </instance>
 <instance part="SUPPLY17" gate="GND" x="190.5" y="154.94" smashed="yes"/>
+<instance part="SUPPLY7" gate="G$1" x="124.46" y="167.64" smashed="yes" rot="R270">
+<attribute name="VALUE" x="127.254" y="167.64" size="1.778" layer="96" rot="R270" align="bottom-center"/>
+</instance>
+<instance part="SUPPLY8" gate="GND" x="114.3" y="162.56" smashed="yes" rot="R90"/>
 </instances>
 <busses>
@@
 </segment>
 <segment>
-<pinref part="SUPPLY8" gate="G$1" pin="VCC"/>
-<pinref part="J4" gate="G$1" pin="2"/>
-<wire x1="124.46" y1="162.56" x2="121.92" y2="162.56" width="0.1524" layer="91"/>
-<pinref part="TP4" gate="G$1" pin="P$1"/>
-<wire x1="121.92" y1="162.56" x2="111.76" y2="162.56" width="0.1524" layer="91"/>
-<junction x="121.92" y="162.56"/>
-</segment>
-<segment>
 <pinref part="C8" gate="G$1" pin="POS"/>
 <pinref part="SUPPLY11" gate="G$1" pin="VCC"/>
@@
 <pinref part="U3" gate="G$1" pin="VIN"/>
 <pinref part="SUPPLY15" gate="G$1" pin="VCC"/>
+</segment>
+<segment>
+<pinref part="J4" gate="G$1" pin="1"/>
+<wire x1="124.46" y1="167.64" x2="119.38" y2="167.64" width="0.1524" layer="91"/>
+<pinref part="TP4" gate="G$1" pin="P$1"/>
+<wire x1="119.38" y1="167.64" x2="111.76" y2="167.64" width="0.1524" layer="91"/>
+<junction x="119.38" y="167.64"/>
+<pinref part="SUPPLY7" gate="G$1" pin="VCC"/>
 </segment>
 </net>
@@
 </segment>
 <segment>
-<pinref part="SUPPLY7" gate="GND" pin="GND"/>
-<pinref part="J4" gate="G$1" pin="1"/>
-<wire x1="124.46" y1="167.64" x2="111.76" y2="167.64" width="0.1524" layer="91"/>
-<pinref part="J4" gate="G$1" pin="3"/>
-<wire x1="111.76" y1="167.64" x2="111.76" y2="165.1" width="0.1524" layer="91"/>
-<junction x="111.76" y="167.64"/>
-</segment>
-<segment>
 <pinref part="C8" gate="G$1" pin="NEG"/>
 <pinref part="SUPPLY12" gate="GND" pin="GND"/>
@@
 <pinref part="SUPPLY17" gate="GND" pin="GND"/>
 </segment>
+<segment>
+<pinref part="J4" gate="G$1" pin="2"/>
+<pinref part="J4" gate="G$1" pin="3"/>
+<wire x1="111.76" y1="165.1" x2="111.76" y2="162.56" width="0.1524" layer="91"/>
+<pinref part="SUPPLY8" gate="GND" pin="GND"/>
+<junction x="111.76" y="162.56"/>
+</segment>
 </net>
